File: chessboard/chessboard.kicad_pcb (KiCad board)
At the start: 2 copper layers, 286 parts, among them J1 Conn_01x08, U1 AMS1117-3.3, U10 MMC5603NJ, U11 PCA9548ADB, U12 MMC5603NJ, U13 MMC5603NJ, U14 MMC5603NJ, U15 MMC5603NJ, U16 MMC5603NJ, U17 MMC5603NJ, U18 MMC5603NJ, U19 MMC5603NJ, U2 PCA9548ADB, U20 PCA9548ADB, U21 MMC5603NJ, U22 MMC5603NJ, U23 MMC5603NJ, U24 MMC5603NJ, U25 MMC5603NJ, U26 MMC5603NJ, U27 MMC5603NJ, U28 MMC5603NJ, U29 PCA9548ADB, U3 MMC5603NJ, U30 MMC5603NJ, U31 MMC5603NJ, U32 MMC5603NJ, U33 MMC5603NJ, U34 MMC5603NJ, U35 MMC5603NJ, U36 MMC5603NJ, U37 MMC5603NJ, U38 PCA9548ADB, U39 MMC5603NJ, U4 MMC5603NJ, U40 MMC5603NJ, U41 MMC5603NJ, U42 MMC5603NJ, U43 MMC5603NJ, U44 MMC5603NJ, U45 MMC5603NJ, U46 MMC5603NJ, U47 PCA9548ADB, U48 MMC5603NJ, U49 MMC5603NJ, U5 MMC5603NJ, U50 MMC5603NJ, U51 MMC5603NJ, U52 MMC5603NJ, U53 MMC5603NJ, U54 MMC5603NJ, U55 MMC5603NJ, U56 PCA9548ADB, U57 MMC5603NJ, U58 MMC5603NJ, U59 MMC5603NJ, U6 MMC5603NJ, U60 MMC5603NJ, U61 MMC5603NJ, U62 MMC5603NJ, U63 MMC5603NJ, U64 MMC5603NJ, U65 PCA9548ADB, U66 MMC5603NJ, U67 MMC5603NJ, U68 MMC5603NJ, U69 MMC5603NJ, U7 MMC5603NJ, U70 MMC5603NJ, U71 MMC5603NJ, U72 MMC5603NJ, U73 MMC5603NJ, U8 MMC5603NJ, U9 MMC5603NJ

Commit message: new single row board
Parts:
- removed C11, C12, C13, C15, C16, C17, C18, C19, C20, C21, C22, C23, C25, C26, C27, C28, C29, C30, C31, C32, C33, C35, C36, C37, C38, C39, C40, C41, C42, C43, C45, C46, C47, C48, C49, C50, C51, C52, C53, C55, C56, C57, C58, C59, C60, C61, C62, C63, C65, C66, C67, C68, C69, C70, C71, C72, C73, C75, C76, C77, C78, C79, C80, C81, C82: 100nF, Capacitor_SMD:C_0805_2012Metric_Pad1.18x1.45mm_HandSolder
- removed C14, C24, C34, C44, C54, C64, C74: 22uF, Capacitor_SMD:C_0805_2012Metric_Pad1.18x1.45mm_HandSolder
- removed D10, D11, D12, D13, D14, D15, D16, D17, D18, D19, D20, D21, D22, D23, D24, D25, D26, D27, D28, D29, D30, D31, D32, D33, D34, D35, D36, D37, D38, D39, D40, D41, D42, D43, D44, D45, D46, D47, D48, D49, D50, D51, D52, D53, D54, D55, D56, D57, D58, D59, D60, D61, D62, D63, D64, D9: WS2812B, LED_SMD:LED_WS2812B_PLCC4_5.0x5.0mm_P3.2mm
- removed J1: Conn_01x08, Connector_JST:JST_PH_B8B-PH-K_1x08_P2.00mm_Vertical
- removed JP10, JP11, JP12, JP13, JP14, JP15, JP16, JP17, JP18, JP19, JP20, JP21, JP22, JP23, JP24, JP25, JP26, JP27, JP28, JP29, JP30, JP31, JP32, JP33, JP5, JP7, JP8, JP9: Jumper_2_Bridged, mylibrary:Bridged 2.5mm 1.0mm Test Points
- removed RN10, RN11, RN12, RN13, RN14, RN15, RN16, RN17, RN18, RN19, RN20, RN21, RN22, RN23, RN24, RN25, RN26, RN27, RN28, RN29, RN30, RN31, RN32, RN33, RN5, RN6, RN7, RN8, RN9: 4.7k, Resistor_SMD:R_Array_Concave_4x0603
- removed U10, U12, U13, U14, U15, U16, U17, U18, U19, U21, U22, U23, U24, U25, U26, U27, U28, U30, U31, U32, U33, U34, U35, U36, U37, U39, U40, U41, U42, U43, U44, U45, U46, U48, U49, U50, U51, U52, U53, U54, U55, U57, U58, U59, U60, U61, U62, U63, U64, U66, U67, U68, U69, U70, U71, U72, U73: MMC5603NJ, Package_BGA:WLP-4_0.86x0.86mm_P0.4mm
- removed U11, U20, U29, U38, U47, U56, U65: PCA9548ADB, Package_SO:SSOP-24_5.3x8.2mm_P0.65mm
- added J2: Conn_01x07, mylibrary:Custom PinSocket Edge Connector, F.Cu at (107.5, 138.8)
- added J3: Conn_01x07, mylibrary:Custom PinSocket Edge Connector, F.Cu at (122.5, 111.2)
- added J4: Conn_01x07, mylibrary:Custom PinSocket Edge Connector, F.Cu at (496.7, 111.2)
- added J5: Conn_01x07, mylibrary:Custom PinSocket Edge Connector, F.Cu at (481.4, 138.8)
- added J6: Conn_01x07, mylibrary:Custom PinSocket Edge Connector, F.Cu at (105.5, 114.0)
- added NT1: NetTie_2, Jumper:SolderJumper-2_P1.3mm_Bridged_Pad1.0x1.5mm, F.Cu at (301.4, 123.2)
- C1, C4: value 22uF -> 100nF
- D1, D2, D3, D4, D5, D6, D7, D8: value WS2812B -> XL-5050RGBC-WS2812B
- JP1: value Jumper_2_Open -> SolderJumper_2_Open; footprint TestPoint:TestPoint_Bridge_Pitch2.54mm_Drill1.0mm -> Resistor_SMD:R_0805_2012Metric_Pad1.20x1.40mm_HandSolder
- JP2, JP3, JP4: value Jumper_2_Bridged -> SolderJumper_3_Open; footprint mylibrary:Bridged 2.5mm 1.0mm Test Points -> Jumper:SolderJumper-3_P2.0mm_Open_TrianglePad1.0x1.5mm
- JP6: value Jumper_2_Bridged -> SolderJumper_2_Open; footprint mylibrary:Bridged 2.5mm 1.0mm Test Points -> Resistor_SMD:R_0805_2012Metric_Pad1.20x1.40mm_HandSolder
- RN1, RN2, RN3, RN4: footprint Resistor_SMD:R_Array_Concave_4x0603 -> Resistor_SMD:R_Array_Convex_4x0603
- U1: value AMS1117-3.3 -> TCA9548APWR; footprint Package_TO_SOT_SMD:SOT-223-3_TabPin2 -> Package_SO:TSSOP-24_4.4x7.8mm_P0.65mm
- U2: value PCA9548ADB -> TMAG5273; footprint Package_SO:SSOP-24_5.3x8.2mm_P0.65mm -> Package_TO_SOT_SMD:SOT-23-6
- U3, U4, U5, U6, U7, U8, U9: value MMC5603NJ -> TMAG5273; footprint Package_BGA:WLP-4_0.86x0.86mm_P0.4mm -> Package_TO_SOT_SMD:SOT-23-6
- moved C2 516.1 mm to (465.5, 134.5)
- moved C1 357.5 mm to (294.0, 120.5), turned to -90 degrees
- moved U1 357.4 mm to (300.4, 112.7), turned to 180 degrees
- moved JP3 333.5 mm to (300.0, 102.5), turned to 180 degrees
- moved JP4 333.5 mm to (300.0, 120.5), turned to 180 degrees
- moved JP2 332.2 mm to (300.0, 105.5), turned to 180 degrees
- moved RN2 252.9 mm to (251.3, 122.2), turned to 90 degrees
- moved RN3 252.9 mm to (351.3, 122.2), turned to 90 degrees
- moved RN4 252.9 mm to (451.3, 122.2), turned to 90 degrees
- moved C4 226.5 mm to (181.0, 125.5)
- moved C6 225.2 mm to (281.0, 125.5), turned to 90 degrees
- moved C8 225.2 mm to (381.0, 125.5), turned to 90 degrees
- moved C5 223.6 mm to (231.0, 125.5), turned to 90 degrees
- moved C7 223.6 mm to (331.0, 125.5), turned to 90 degrees
- moved C10 215.6 mm to (470.0, 126.0), turned to 90 degrees
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Connections:
- C1 pad 1: +5V -> +3.3V
- C2 pad 1: +3.3V -> +5V
- C4 pad 1: +5V -> +3.3V
- D8 pad 2: /Row0/LED_OUT -> /LED_OUT
- JP1 pad 1: Net-(J1-Pin_5) -> /LED_OUT
- JP2 pad 1: +3.3V -> GND
- JP2 pad 2: Net-(JP2-B) -> Net-(JP2-C)
- JP3 pad 2: Net-(JP3-B) -> Net-(JP3-C)
- JP4 pad 2: Net-(JP4-B) -> Net-(JP4-C)
- JP6 pad 1: +3.3V -> /LED_IN
- JP6 pad 2: Net-(JP6-B) -> /LED_RET
- RN1 pad 5: unconnected-(RN1-R4.2-Pad5) -> /Row0/sensorpair3/C1
- RN1 pad 6: /SDA -> /Row0/sensorpair3/D1
- RN1 pad 7: unconnected-(RN1-R2.2-Pad7) -> /Row0/sensorpair3/C0
- RN1 pad 8: /SCL -> /Row0/sensorpair3/D0
- RN2 pad 5: /Row0/sensorpair0/C1 -> /Row0/sensorpair2/C1
- RN2 pad 6: /Row0/sensorpair0/D1 -> /Row0/sensorpair2/D1
- RN2 pad 7: /Row0/sensorpair0/C0 -> /Row0/sensorpair2/C0
- RN2 pad 8: /Row0/sensorpair0/D0 -> /Row0/sensorpair2/D0
- RN3 pad 5: /Row0/sensorpair1/C1 -> /Row0/sensorpair0/C1
- RN3 pad 6: /Row0/sensorpair1/D1 -> /Row0/sensorpair0/D1
- RN3 pad 7: /Row0/sensorpair1/C0 -> /Row0/sensorpair0/C0
- RN3 pad 8: /Row0/sensorpair1/D0 -> /Row0/sensorpair0/D0
- RN4 pad 5: /Row0/sensorpair2/C1 -> /Row0/sensorpair1/C1
- RN4 pad 6: /Row0/sensorpair2/D1 -> /Row0/sensorpair1/D1
- RN4 pad 7: /Row0/sensorpair2/C0 -> /Row0/sensorpair1/C0
- RN4 pad 8: /Row0/sensorpair2/D0 -> /Row0/sensorpair1/D0
- U1 pad 1: GND -> Net-(JP4-C)
- U1 pad 2: +3.3V -> Net-(JP2-C)
- U1 pad 3: +5V -> Net-(U1-~{RESET})
- U2 pad 1: Net-(JP5-B) -> /Row0/sensorpair3/C0
- U2 pad 2: Net-(JP4-B) -> GND
- U2 pad 3: Net-(JP2-B) -> GND
- U2 pad 4: /Row0/sensorpair0/D0 -> +3.3V
- U2 pad 5: /Row0/sensorpair0/C0 -> GND
- U2 pad 6: /Row0/sensorpair0/D1 -> /Row0/sensorpair3/D0
Routing:
- net +3.3V: track 5074.1 -> 552.5 mm, vias 0 -> 5
- net +5V: track 3403.8 -> 452.1 mm
- net /Row7/sensorpair3/C1: track 439.8 -> 0.00 mm, vias 2 -> 0
- net /Row5/sensorpair3/C1: track 439.8 -> 0.00 mm, vias 2 -> 0
- net /Row4/sensorpair3/C1: track 439.8 -> 0.00 mm, vias 2 -> 0
- net /Row3/sensorpair3/C1: track 439.8 -> 0.00 mm, vias 2 -> 0
- net /Row2/sensorpair3/C1: track 439.8 -> 0.00 mm, vias 2 -> 0
- net /Row1/sensorpair3/C1: track 439.8 -> 0.00 mm, vias 2 -> 0
- net /Row6/sensorpair3/C1: track 439.8 -> 0.00 mm, vias 2 -> 0
- net /Row7/sensorpair3/D1: track 431.3 -> 0.00 mm, vias 2 -> 0
- net /Row6/sensorpair3/D1: track 431.3 -> 0.00 mm, vias 2 -> 0
- net /Row5/sensorpair3/D1: track 431.3 -> 0.00 mm, vias 2 -> 0
- net /Row4/sensorpair3/D1: track 431.3 -> 0.00 mm, vias 2 -> 0
- net /Row3/sensorpair3/D1: track 431.3 -> 0.00 mm, vias 2 -> 0
- net /Row2/sensorpair3/D1: track 431.3 -> 0.00 mm, vias 2 -> 0
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- added copper zone on B.Cu, net GND
Other:
- board outline added: 400 x 50 mm
- board text added: "0"
- board text added: "1"
- board text added: "JLCJLCJLCJLC"
- board text added: "LED Out & Ret Loop"
- board text added: "LED Ret & IN"
- board text removed: "todo: move drawings to silkscreen"

Commit message: make it pretty
Parts:
- added G***: LOGO, LOGO, F.Cu at (175.0, 109.0)
- added H1: MountingHole_Pad, MountingHole:MountingHole_3.2mm_M3_ISO14580_Pad, F.Cu at (489.8, 120.0)
- added H2: MountingHole_Pad, MountingHole:MountingHole_3.2mm_M3_ISO14580_Pad, F.Cu at (140.0, 120.0)
- added H3: MountingHole_Pad, MountingHole:MountingHole_3.2mm_M3_ISO14580_Pad, F.Cu at (310.0, 140.0)
- moved JP1 1.75 mm to (112.0, 133.8)
- moved U1 0.40 mm to (300.0, 112.7)
Routing:
- net Net-(JP2-C): track 12.7 -> 10.8 mm
- net /LED_OUT: track 396.0 -> 397.8 mm
- net GND: track 498.9 -> 500.1 mm
- net Net-(JP4-C): track 5.88 -> 7.03 mm
- net /Row0/sensorpair1/D0: track 154.0 -> 155.2 mm
- net /Row0/sensorpair0/D0: track 56.9 -> 58.0 mm
- net Net-(U1-~{RESET}): track 12.0 -> 13.1 mm
- net /Row0/sensorpair1/D1: track 197.8 -> 198.9 mm
- net /Row0/sensorpair1/C1: track 205.8 -> 207.0 mm
- net /Row0/sensorpair0/D1: track 89.8 -> 91.0 mm
- net /Row0/sensorpair0/C1: track 92.8 -> 93.9 mm
- net /Row0/sensorpair0/C0: track 66.0 -> 67.1 mm
- net /Row0/sensorpair1/C0: track 164.4 -> 165.5 mm
Other:
- board text added: "+3V3"
- board text added: "+5V"
- board text added: "A"
- board text added: "B"
- board text added: "C"
- board text added: "ChessBoard Segment"
- board text added: "D"
- board text added: "Designed by Karmanyaah Malhotra Feb 2024"
- board text added: "E"
- board text added: "F"
- board text added: "For UT Austin IEEE RAS https://github.com/ut-ras/chessbot"
- board text added: "G"
- board text added: "GND"
- board text added: "GND/M3"
- board text added: "H"
- board text added: "LED_IN"
- board text added: "LED_OUT"
- board text added: "LED_RET"
- board text added: "Ret/In Jumper is a test point only"
- board text added: "SCL"
- board text added: "SDA"
- board text added: "Solder Out/Ret jumper on last board"
- board text added: "U2-9 TMAG5273 SOT-23-6 U1 TCA9548APWR TSSOP-24_4.4x7.8mm_P0.65mm RN1-4 4.7kΩ 4x0603 D1-8 WS2812B WS2812B C2 ~22uF 0805_Handsolder (so 0603 or 0805) C1,3-10 ~100nF 0805_Handsolder (so 0603 or 0805) Board2Board Connectors - whatever you like (2.54mm Pin Spacing)"
- board text added: "locked"

Commit message: ready to buy
Parts:
- removed NT1: NetTie_2, Jumper:SolderJumper-2_P1.3mm_Bridged_Pad1.0x1.5mm
- added JP5: SolderJumper_2_Open, Jumper:SolderJumper-2_P1.3mm_Open_Pad1.0x1.5mm, F.Cu at (306.2, 123.8)
- added R1: 10k, Resistor_SMD:R_0805_2012Metric_Pad1.20x1.40mm_HandSolder, F.Cu at (302.2, 123.8)
Routing:
- net /Row0/sensorpair3/D1: track 165.4 -> 161.1 mm
- net GND: track 500.1 -> 503.3 mm
- net /LED_RET: track 47.3 -> 44.2 mm
- net /SCL: track 243.8 -> 241.2 mm
- net /SDA: track 244.1 -> 241.7 mm
- net /LED_IN: track 44.6 -> 42.2 mm
- net +3.3V: track 552.5 -> 550.1 mm
- net Net-(JP5-B): track 13.1 -> 15.4 mm
- net /LED_OUT: track 397.8 -> 396.6 mm
- net +5V: track 452.1 -> 451.3 mm
- added copper zone on F.Cu, net +5V
- added copper zone on F.Cu, net GND
