File: controlboard/Power.kicad_sch (KiCad schematic)
At the start: 35 parts, among them J11 Pololu Voltage Regulator, J4 USB_C_Receptacle_USB2.0_14P, J7 Screw_Terminal_01x02, J9 mini560 voltage regulator, Q2 PMOS AO3401A, U4 CH224K

Commit message: erc should be good now
Parts:
- U4: footprint 0chessbot-parts:SSOP-10-1EP_3.9x4.9mm_P1mm_EP2.1x3.3mm -> 0my_project:ESSOP-10_CH224K
Connections:
- net at J4.A5 (CC1), TP12.1: now also U4.4 (DP); no longer U4.7 (CC1)
- net at J4.A6 (D+), J4.B6 (D+): now also U4.6 (CC2); no longer U4.4 (DP)
- net at J4.A7 (D-), J4.B7 (D-): now also U4.7 (CC1); no longer U4.5 (DM)
- net at J4.B5 (CC2), TP13.1: now also U4.5 (DM); no longer U4.6 (CC2)
Changed lines of the file:
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@@
 	(paper "A4")
 	(junction
-		(at 46.99 45.72)
+		(at 93.98 113.03)
 		(diameter 0)
 		(color 0 0 0 0)
@@
 	)
 	(junction
+		(at 48.26 19.05)
+		(diameter 0)
+		(color 0 0 0 0)
+	)
+	(junction
 		(at 53.34 19.05)
 		(diameter 0)
@@
 	)
 	(junction
-		(at 93.98 113.665)
-		(diameter 0)
-		(color 0 0 0 0)
-	)
-	(junction
 		(at 85.09 58.42)
 		(diameter 0)
@@
 		(color 0 0 0 0)
 	)
+	(junction
+		(at 46.99 44.45)
+		(diameter 0)
+		(color 0 0 0 0)
+	)
 	(no_connect
 		(at 229.87 35.56)
@@
 	(wire
 		(pts
+			(xy 66.04 46.99) (xy 66.04 48.26)
+		)
+		(stroke
+			(width 0)
+			(type default)
+		)
+	)
+	(wire
+		(pts
 			(xy 60.96 24.13) (xy 62.23 24.13)
 		)
@@
 	(wire
 		(pts
+			(xy 93.98 114.3) (xy 93.98 113.03)
+		)
+		(stroke
+			(width 0)
+			(type default)
+		)
+	)
+	(wire
+		(pts
 			(xy 237.49 33.02) (xy 236.22 33.02)
 		)
@@
 	(wire
 		(pts
-			(xy 46.99 45.72) (xy 66.04 45.72)
+			(xy 46.99 44.45) (xy 66.04 44.45)
 		)
 		(stroke
@@
 	(wire
 		(pts
-			(xy 93.98 115.57) (xy 107.95 115.57)
+			(xy 93.98 114.3) (xy 107.95 114.3)
 		)
 		(stroke
@@
 	(wire
 		(pts
-			(xy 93.98 113.665) (xy 93.98 115.57)
-		)
-		(stroke
-			(width 0)
-			(type default)
-		)
-	)
-	(wire
-		(pts
 			(xy 180.34 45.72) (xy 181.61 45.72)
 		)
@@
 	(wire
 		(pts
-			(xy 46.99 19.05) (xy 53.34 19.05)
+			(xy 46.99 19.05) (xy 48.26 19.05)
 		)
 		(stroke
@@
 	(wire
 		(pts
-			(xy 93.98 111.76) (xy 93.98 113.665)
+			(xy 93.98 111.76) (xy 93.98 113.03)
 		)
 		(stroke
@@
 	(wire
 		(pts
+			(xy 46.99 44.45) (xy 46.99 45.72)
+		)
+		(stroke
+			(width 0)
+			(type default)
+		)
+	)
+	(wire
+		(pts
 			(xy 85.09 50.8) (xy 85.09 44.45)
 		)
@@
 	(wire
 		(pts
-			(xy 46.99 43.18) (xy 46.99 45.72)
+			(xy 46.99 43.18) (xy 46.99 44.45)
 		)
 		(stroke
@@
 	(wire
 		(pts
+			(xy 48.26 19.05) (xy 53.34 19.05)
+		)
+		(stroke
+			(width 0)
+			(type default)
+		)
+	)
+	(wire
+		(pts
 			(xy 85.09 44.45) (xy 83.82 44.45)
 		)
@@
 	(hierarchical_label "SERVO_5V"
 		(shape input)
-		(at 107.95 115.57 0)
+		(at 107.95 114.3 0)
 		(fields_autoplaced yes)
 		(effects
@@
 	)
 	(symbol
+		(lib_id "power:PWR_FLAG")
+		(at 48.26 19.05 0)
+		(unit 1)
+		(exclude_from_sim no)
+		(in_bom yes)
+		(on_board yes)
+		(dnp no)
+		(fields_autoplaced yes)
+		(property "Reference" "#FLG01"
+			(at 48.26 17.145 0)
+			(effects
+				(font
+					(size 1.27 1.27)
+				)
+				(hide yes)
+			)
+		)
+		(property "Value" "PWR_FLAG"
+			(at 48.26 13.97 0)
+			(effects
+				(font
+					(size 1.27 1.27)
+				)
+			)
+		)
+		(property "Footprint" ""
+			(at 48.26 19.05 0)
+			(effects
+				(font
+					(size 1.27 1.27)
+				)
+				(hide yes)
+			)
+		)
+		(property "Datasheet" "~"
+			(at 48.26 19.05 0)
+			(effects
+				(font
+					(size 1.27 1.27)
+				)
+				(hide yes)
+			)
+		)
+		(property "Description" "Special symbol for telling ERC where power comes from"
+			(at 48.26 19.05 0)
+			(effects
+				(font
+					(size 1.27 1.27)
+				)
+				(hide yes)
+			)
+		)
+		(pin "1"
+		)
+		(instances
+			(project "controlboard"
+				(path "/2797250d-6fee-4769-b4dd-0e20ce4f0941/5fab4b81-761e-4fae-b113-00364a75fd9a"
+					(reference "#FLG01")
+					(unit 1)
+				)
+			)
+		)
+	)
+	(symbol
 		(lib_id "Jumper:SolderJumper_2_Open")
 		(at 92.71 54.61 90)
@@
 			)
 		)
-		(property "Description" ""
+		(property "Description" "Power symbol creates a global label with name \"GND\" , ground"
 			(at 255.27 76.2 0)
 			(effects
@@
 			)
 		)
-		(property "Description" ""
+		(property "Description" "Power symbol creates a global label with name \"GND\" , ground"
 			(at 240.03 76.2 0)
 			(effects
@@
 			)
 		)
-		(property "Footprint" "0chessbot-parts:SSOP-10-1EP_3.9x4.9mm_P1mm_EP2.1x3.3mm"
+		(property "Footprint" "0my_project:ESSOP-10_CH224K"
 			(at 92.71 60.96 0)
 			(effects
@@
 		)
 		(pin "OUT" input
-			(at 93.98 113.665 0)
+			(at 93.98 113.03 0)
 			(effects
 				(font

Commit message: pcb layout work
Parts:
- TP11, TP12, TP13, TP14: footprint Connector_PinSocket_2.54mm:PinSocket_1x01_P2.54mm_Vertical -> TestPoint:TestPoint_THTPad_1.0x1.0mm_Drill0.5mm
- U4: footprint 0my_project:ESSOP-10_CH224K -> 0chessbot-parts:SSOP-10-1EP_3.9x4.9mm_P1mm_EP2.1x3.3mm
Connections:
- net GND: now also U4.11 (GND); no longer U4.0 (GND)
- net at J4.A5 (CC1), TP12.1: now also U4.7 (CC1); no longer U4.4 (DP)
- net at J4.A6 (D+), J4.B6 (D+): now also U4.4 (DP); no longer U4.6 (CC2)
- net at J4.A7 (D-), J4.B7 (D-): now also U4.5 (DM); no longer U4.7 (CC1)
- net at J4.B5 (CC2), TP13.1: now also U4.6 (CC2); no longer U4.5 (DM)
Changed lines of the file:
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@@
 	(paper "A4")
 	(junction
+		(at 46.99 45.72)
+		(diameter 0)
+		(color 0 0 0 0)
+	)
+	(junction
 		(at 93.98 113.03)
 		(diameter 0)
@@
 		(color 0 0 0 0)
 	)
-	(junction
-		(at 46.99 44.45)
-		(diameter 0)
-		(color 0 0 0 0)
-	)
 	(no_connect
 		(at 229.87 35.56)
@@
 	(wire
 		(pts
-			(xy 66.04 46.99) (xy 66.04 48.26)
-		)
-		(stroke
-			(width 0)
-			(type default)
-		)
-	)
-	(wire
-		(pts
 			(xy 60.96 24.13) (xy 62.23 24.13)
 		)
@@
 	(wire
 		(pts
-			(xy 46.99 44.45) (xy 66.04 44.45)
+			(xy 46.99 45.72) (xy 66.04 45.72)
 		)
 		(stroke
@@
 	(wire
 		(pts
+			(xy 46.99 43.18) (xy 46.99 45.72)
+		)
+		(stroke
+			(width 0)
+			(type default)
+		)
+	)
+	(wire
+		(pts
 			(xy 31.75 69.85) (xy 31.75 68.58)
 		)
@@
 	(wire
 		(pts
-			(xy 46.99 44.45) (xy 46.99 45.72)
-		)
-		(stroke
-			(width 0)
-			(type default)
-		)
-	)
-	(wire
-		(pts
 			(xy 85.09 50.8) (xy 85.09 44.45)
 		)
@@
 	(wire
 		(pts
-			(xy 46.99 43.18) (xy 46.99 44.45)
-		)
-		(stroke
-			(width 0)
-			(type default)
-		)
-	)
-	(wire
-		(pts
 			(xy 243.84 135.89) (xy 245.11 135.89)
 		)
@@
 			)
 		)
-		(property "Footprint" "Connector_PinSocket_2.54mm:PinSocket_1x01_P2.54mm_Vertical"
+		(property "Footprint" "TestPoint:TestPoint_THTPad_1.0x1.0mm_Drill0.5mm"
 			(at 67.31 24.13 0)
 			(effects
@@
 			)
 		)
-		(property "Footprint" "Connector_PinSocket_2.54mm:PinSocket_1x01_P2.54mm_Vertical"
+		(property "Footprint" "TestPoint:TestPoint_THTPad_1.0x1.0mm_Drill0.5mm"
 			(at 58.42 38.1 0)
 			(effects
@@
 			)
 		)
-		(property "Footprint" "0my_project:ESSOP-10_CH224K"
+		(property "Footprint" "0chessbot-parts:SSOP-10-1EP_3.9x4.9mm_P1mm_EP2.1x3.3mm"
 			(at 92.71 60.96 0)
 			(effects
@@
 		(pin "3"
 		)
-		(pin "0"
+		(pin "11"
 		)
 		(pin "5"
@@
 			)
 		)
-		(property "Footprint" "Connector_PinSocket_2.54mm:PinSocket_1x01_P2.54mm_Vertical"
+		(property "Footprint" "TestPoint:TestPoint_THTPad_1.0x1.0mm_Drill0.5mm"
 			(at 58.42 19.05 0)
 			(effects
@@
 			)
 		)
-		(property "Footprint" "Connector_PinSocket_2.54mm:PinSocket_1x01_P2.54mm_Vertical"
+		(property "Footprint" "TestPoint:TestPoint_THTPad_1.0x1.0mm_Drill0.5mm"
 			(at 55.88 35.56 0)
 			(effects
