File: controlboard/controlboard.kicad_pcb (KiCad board)
At the start: 2 copper layers, 5 parts

Commit message: Control Board major progress
Parts:
- removed the REF** at (94.5, 78.4)
- added J1: GPIO, Connector_PinSocket_2.54mm:PinSocket_2x20_P2.54mm_Vertical, B.Cu at (192.7, 62.4)
- added REF**: BarrelJack_CUI_PJ-063AH_Horizontal, Connector_BarrelJack:BarrelJack_CUI_PJ-063AH_Horizontal, F.Cu at (129.8, 32.0)
- added REF**: USB_C_Receptacle_GCT_USB4105-xx-A_16P_TopMnt_Horizontal, Connector_USB:USB_C_Receptacle_GCT_USB4105-xx-A_16P_TopMnt_Horizontal, F.Cu at (105.0, 24.2)
- moved REF** 105.0 mm to (93.9, 26.2)
- moved REF** 34.6 mm to (122.0, 78.7)
- moved REF** 31.3 mm to (122.4, 51.6)
Other:
- board outline added: 130.3 x 93.6 mm
- board text added: "CAMERA (OPTIONAL)"
- board text added: "DISPLAY (OPTIONAL)"
- board text added: "Extend PCB edge 0.5mm if using SMT header"
- board text added: "PoE"
- board text added: "RJ45"
- board text added: "USB"

Commit message: more progress on controlboard pcb
Parts:
- removed the REF** at (89.5, 43.8)
- removed the REF** at (93.9, 26.2)
- added J1 (x2): GPIO, Connector_PinSocket_2.54mm:PinSocket_2x20_P2.54mm_Vertical, B.Cu at (108.2, 48.8)
- added J1: GPIO, Connector_PinSocket_2.54mm:PinSocket_2x20_P2.54mm_Vertical, B.Cu at (26.6, 42.0)
- added MH1: MountingHole_2.7mm_M2.5, MountingHole:MountingHole_2.7mm_M2.5, F.Cu at (21.8, 40.8)
- added MH1 (x2): MountingHole_2.7mm_M2.5, MountingHole:MountingHole_2.7mm_M2.5, F.Cu at (103.4, 47.5)
- added MH2 (x2): MountingHole_2.7mm_M2.5, MountingHole:MountingHole_2.7mm_M2.5, F.Cu at (161.4, 47.5)
- added MH2: MountingHole_2.7mm_M2.5, MountingHole:MountingHole_2.7mm_M2.5, F.Cu at (79.8, 40.8)
- added MH3: MountingHole_2.7mm_M2.5, MountingHole:MountingHole_2.7mm_M2.5, F.Cu at (21.8, 63.8)
- added MH3: MountingHole_2.7mm_M2.5, MountingHole:MountingHole_2.7mm_M2.5, F.Cu at (103.4, 96.5)
- added MH3: MountingHole_2.7mm_M2.5, MountingHole:MountingHole_2.7mm_M2.5, F.Cu at (103.4, 70.5)
- added MH4: MountingHole_2.7mm_M2.5, MountingHole:MountingHole_2.7mm_M2.5, F.Cu at (161.4, 70.5)
- added MH4: MountingHole_2.7mm_M2.5, MountingHole:MountingHole_2.7mm_M2.5, F.Cu at (79.8, 63.8)
- added MH4: MountingHole_2.7mm_M2.5, MountingHole:MountingHole_2.7mm_M2.5, F.Cu at (161.4, 96.5)
- added REF**: PinSocket_2x20_P2.54mm_Vertical_SMD, Connector_PinSocket_2.54mm:PinSocket_2x20_P2.54mm_Vertical_SMD, F.Cu at (132.4, 47.5)
- added REF**: SolderJumper-2_P1.3mm_Open_Pad1.0x1.5mm, Jumper:SolderJumper-2_P1.3mm_Open_Pad1.0x1.5mm, F.Cu at (124.0, 82.8)
- added REF**: PinSocket_2x20_P2.54mm_Horizontal, Connector_PinSocket_2.54mm:PinSocket_2x20_P2.54mm_Horizontal, F.Cu at (108.1, 94.9)
- added REF**: SolderJumper-2_P1.3mm_Open_Pad1.0x1.5mm, Jumper:SolderJumper-2_P1.3mm_Open_Pad1.0x1.5mm, F.Cu at (124.0, 80.8)
- added REF**: SolderJumper-2_P1.3mm_Open_Pad1.0x1.5mm, Jumper:SolderJumper-2_P1.3mm_Open_Pad1.0x1.5mm, F.Cu at (124.0, 78.8)
- added REF**: R_0603_1608Metric_Pad0.98x0.95mm_HandSolder, Resistor_SMD:R_0603_1608Metric_Pad0.98x0.95mm_HandSolder, F.Cu at (124.0, 84.8)
- moved J1 68.9 mm to (260.9, 52.5)
- moved REF** 56.6 mm to (106.8, 83.8), turned to -90 degrees
- moved REF** 42.1 mm to (142.4, 88.7), turned to 90 degrees
- moved REF** 33.0 mm to (103.5, 57.2), turned to -90 degrees
- moved REF** 9.99 mm to (122.1, 88.7), turned to 90 degrees
Other:
- board size 130.3 x 93.6 mm -> 319.5 x 172 mm
- board text added: "4mm clearance (incl.)"
- board text added: "5mm clearance (incl.)"
- board text added: "6mm clearance (incl. 1 safety)"
- board text added: "B,G,R,Y, etc, etc todo"
- board text added: "ChBoard"
- board text added: "Lim Switches"
- board text added: "Motor1 Motor2"
- board text added: "Pwr"
- board text added: "SD Card clearance"
- board text added: "Srvo"

Commit message: ControlBoard Schematic nearly done
Parts:
- removed the J1 at (108.2, 48.8)
- removed the J1 at (260.9, 52.5)
- removed the REF** at (124.0, 82.8)
- removed the REF** at (122.1, 88.7)
- removed the REF** at (124.0, 80.8)
- removed the REF** at (124.0, 78.8)
- removed the REF** at (142.4, 88.7)
- added A1: Pololu_Breakout_MP6500, Module:Pololu_Breakout-16_15.2x20.3mm, F.Cu at (119.0, 85.4)
- added A2: SilentStepStick TMC5160T, Module:Pololu_Breakout-16_15.2x20.3mm, F.Cu at (139.8, 85.4)
- added C1: 100u, Capacitor_SMD:CP_Elec_6.3x5.4, F.Cu at (109.9, 15.4)
- added C10: 100u, Capacitor_SMD:CP_Elec_6.3x5.4, F.Cu at (139.8, 25.6)
- added C11: 100n, Capacitor_SMD:C_0603_1608Metric_Pad1.08x0.95mm_HandSolder, F.Cu at (293.2, 22.4)
- added C12: 22uF, Capacitor_SMD:C_1206_3216Metric_Pad1.33x1.80mm_HandSolder, F.Cu at (237.3, -8.11)
- added C13: 100n, Capacitor_SMD:C_0603_1608Metric_Pad1.08x0.95mm_HandSolder, F.Cu at (293.2, 42.0)
- added C14: 22uF, Capacitor_SMD:C_1206_3216Metric_Pad1.33x1.80mm_HandSolder, F.Cu at (237.3, -5.60)
- added C2: 100n, Capacitor_SMD:C_0603_1608Metric_Pad1.08x0.95mm_HandSolder, F.Cu at (245.5, -2.19)
- added C3: 22uF, Capacitor_SMD:C_1206_3216Metric_Pad1.33x1.80mm_HandSolder, F.Cu at (125.8, 13.1)
- added C4: 22uF, Capacitor_SMD:C_1206_3216Metric_Pad1.33x1.80mm_HandSolder, F.Cu at (125.8, 16.4)
- added C5: 1u, Capacitor_SMD:C_0603_1608Metric_Pad1.08x0.95mm_HandSolder, F.Cu at (237.3, -10.6)
- added C6: 22uF, Capacitor_SMD:C_1206_3216Metric_Pad1.33x1.80mm_HandSolder, F.Cu at (212.9, 4.03)
- added C7: 22uF, Capacitor_SMD:C_1206_3216Metric_Pad1.33x1.80mm_HandSolder, F.Cu at (219.2, 4.03)
- added C8: 100n, Capacitor_SMD:C_0603_1608Metric_Pad1.08x0.95mm_HandSolder, F.Cu at (123.0, 55.1)
- added C9: 22uF, Capacitor_SMD:C_1206_3216Metric_Pad1.33x1.80mm_HandSolder, F.Cu at (225.6, 4.03)
- added D1: SM4007PL, Diode_SMD:Nexperia_CFP3_SOD-123W, F.Cu at (118.1, 23.1)
- added D10: Y, LED_SMD:LED_0603_1608Metric_Pad1.05x0.95mm_HandSolder, F.Cu at (278.5, -1.70)
- added D11: G, LED_SMD:LED_0603_1608Metric_Pad1.05x0.95mm_HandSolder, F.Cu at (245.5, 13.0)
- added D12: R, LED_SMD:LED_0603_1608Metric_Pad1.05x0.95mm_HandSolder, F.Cu at (245.5, 15.6)
- added D13: G, LED_SMD:LED_0603_1608Metric_Pad1.05x0.95mm_HandSolder, F.Cu at (245.5, 18.2)
- added D14: WS2812B, LED_SMD:LED_WS2812B_PLCC4_5.0x5.0mm_P3.2mm, F.Cu at (231.6, 51.9)
- added D15: WS2812B, LED_SMD:LED_WS2812B_PLCC4_5.0x5.0mm_P3.2mm, F.Cu at (231.6, 58.5)
- added D16: 20V+ D_TVS, Diode_SMD:D_SOD-123F, F.Cu at (118.0, 13.1)
- added D17: 3V3V+ D_TVS, Diode_SMD:D_SOD-123F, F.Cu at (118.0, 16.4)
- added D18: 6V+ D_TVS, Diode_SMD:D_SOD-123F, F.Cu at (118.0, 19.8)
- added D2: Y, LED_SMD:LED_0603_1608Metric_Pad1.05x0.95mm_HandSolder, F.Cu at (278.5, -6.88)
- added D20: R, LED_SMD:LED_0603_1608Metric_Pad1.05x0.95mm_HandSolder, F.Cu at (119.6, 58.0)
- added D21: R, LED_SMD:LED_0603_1608Metric_Pad1.05x0.95mm_HandSolder, F.Cu at (301.9, 29.0)
- added D22: G, LED_SMD:LED_0603_1608Metric_Pad1.05x0.95mm_HandSolder, F.Cu at (245.5, 20.8)
- added D23: G, LED_SMD:LED_0603_1608Metric_Pad1.05x0.95mm_HandSolder, F.Cu at (119.6, 60.6)
- added D25: G, LED_SMD:LED_0603_1608Metric_Pad1.05x0.95mm_HandSolder, F.Cu at (301.9, 31.6)
- added D26: G, LED_SMD:LED_0603_1608Metric_Pad1.05x0.95mm_HandSolder, F.Cu at (245.5, 23.4)
- added D27: G, LED_SMD:LED_0603_1608Metric_Pad1.05x0.95mm_HandSolder, F.Cu at (245.5, 25.9)
- added D28: R, LED_SMD:LED_0603_1608Metric_Pad1.05x0.95mm_HandSolder, F.Cu at (245.5, 28.5)
- added D29: SS54, Diode_SMD:D_SMA_Handsoldering, F.Cu at (284.1, -23.0)
- added D3: Y, LED_SMD:LED_0603_1608Metric_Pad1.05x0.95mm_HandSolder, F.Cu at (278.5, -4.29)
- added D30: SS54, Diode_SMD:D_SMA_Handsoldering, F.Cu at (294.8, -23.0)
- added D31: R, LED_SMD:LED_0603_1608Metric_Pad1.05x0.95mm_HandSolder, F.Cu at (301.9, 48.6)
- added D32: G, LED_SMD:LED_0603_1608Metric_Pad1.05x0.95mm_HandSolder, F.Cu at (301.9, 51.2)
- added D4: G, LED_SMD:LED_0603_1608Metric_Pad1.05x0.95mm_HandSolder, F.Cu at (245.5, 10.4)
- added D5: SM4007PL, Diode_SMD:Nexperia_CFP3_SOD-123W, F.Cu at (118.1, 26.3)
- added D6: WS2812B, LED_SMD:LED_WS2812B_PLCC4_5.0x5.0mm_P3.2mm, F.Cu at (231.6, 38.6)
- added D7: WS2812B, LED_SMD:LED_WS2812B_PLCC4_5.0x5.0mm_P3.2mm, F.Cu at (231.6, 45.2)
- added D8: SM4007PL, Diode_SMD:Nexperia_CFP3_SOD-123W, F.Cu at (206.2, 4.25)
- added J1: Conn_02x04_Counter_Clockwise, Connector_PinSocket_2.54mm:PinSocket_2x04_P2.54mm_Horizontal, F.Cu at (148.9, 94.0)
- added J11: Pololu Voltage Regulator, 0chessbot-parts:reg15d, F.Cu at (132.5, 52.6)
- added J2: Conn_02x04_Row_Letter_Last, Connector_PinSocket_2.54mm:PinSocket_2x04_P2.54mm_Horizontal, F.Cu at (128.6, 94.0)
- added J27: GPIO, Connector_PinSocket_2.54mm:PinSocket_2x20_P2.54mm_Vertical_SMD, F.Cu at (132.4, 47.5)
- added J3: Conn_02x04_Counter_Clockwise, Connector_PinSocket_2.54mm:PinSocket_2x04_P2.54mm_Horizontal, F.Cu at (138.8, 94.0)
- added J4: USB_C_Receptacle_USB2.0_14P, Connector_USB:USB_C_Receptacle_HRO_TYPE-C-31-M-12, B.Cu at (102.6, 58.0)
- added J5: Conn_02x04_Row_Letter_First, Connector_PinSocket_2.54mm:PinSocket_2x04_P2.54mm_Horizontal, F.Cu at (118.3, 94.0)
- added J6: Conn_02x04_Counter_Clockwise, Connector_PinSocket_2.54mm:PinSocket_2x04_P2.54mm_Horizontal, F.Cu at (107.8, 94.0)
- added J7: Screw_Terminal_01x02, TerminalBlock_RND:TerminalBlock_RND_205-00287_1x02_P5.08mm_Horizontal, F.Cu at (226.5, -5.55)
- added J8: Conn_01x02_Pin, Connector_PinHeader_2.54mm:PinHeader_1x02_P2.54mm_Vertical, F.Cu at (252.4, 62.1)
- added J9: mini560 voltage regulator, 0chessbot-parts:mini560, F.Cu at (157.9, 70.5)
- added J??: GPIO, Connector_PinSocket_2.54mm:PinSocket_2x20_P2.54mm_Vertical, B.Cu at (387.5, 31.7)
- added J?? (x2): GPIO, Connector_PinSocket_2.54mm:PinSocket_2x20_P2.54mm_Vertical, B.Cu at (397.7, 116.4)
- added JP1: SolderJumper_2_Bridged, Jumper:SolderJumper-2_P1.3mm_Bridged2Bar_RoundedPad1.0x1.5mm, F.Cu at (238.0, 37.1)
- added JP10: SolderJumper_2_Bridged, Jumper:SolderJumper-2_P1.3mm_Bridged2Bar_RoundedPad1.0x1.5mm, F.Cu at (109.2, 77.0)
- added JP11: SolderJumper_2_Open, Jumper:SolderJumper-2_P1.3mm_Open_RoundedPad1.0x1.5mm, F.Cu at (238.0, 47.7)
- added JP12: SolderJumper_2_Open, Jumper:SolderJumper-2_P1.3mm_Open_RoundedPad1.0x1.5mm, F.Cu at (238.0, 51.3)
- added JP13: Jumper_2_Bridged, TestPoint:TestPoint_2Pads_Pitch2.54mm_Drill0.8mm, F.Cu at (274.9, 20.8)
- added JP14: Jumper_2_Bridged, TestPoint:TestPoint_2Pads_Pitch2.54mm_Drill0.8mm, F.Cu at (274.9, 24.2)
- added JP15: Jumper_2_Bridged, TestPoint:TestPoint_2Pads_Pitch2.54mm_Drill0.8mm, F.Cu at (274.9, 27.5)
- added JP16: Jumper_2_Bridged, TestPoint:TestPoint_2Pads_Pitch2.54mm_Drill0.8mm, F.Cu at (274.9, 30.9)
- added JP17: Jumper_2_Bridged, TestPoint:TestPoint_2Pads_Pitch2.54mm_Drill0.8mm, F.Cu at (274.9, 34.2)
- added JP18: SolderJumper_2_Open, Jumper:SolderJumper-2_P1.3mm_Open_RoundedPad1.0x1.5mm, F.Cu at (238.0, 54.8)
- added JP19: SolderJumper_2_Open, Jumper:SolderJumper-2_P1.3mm_Open_RoundedPad1.0x1.5mm, F.Cu at (238.0, 58.4)
- added JP2: SolderJumper_3_Bridged12, Jumper:SolderJumper-3_P1.3mm_Bridged12_RoundedPad1.0x1.5mm, F.Cu at (109.3, 89.4)
- added JP20: SolderJumper_2_Bridged, Jumper:SolderJumper-2_P1.3mm_Bridged2Bar_RoundedPad1.0x1.5mm, F.Cu at (109.2, 80.6)
- added JP21: Bypass, Jumper:SolderJumper-2_P1.3mm_Open_RoundedPad1.0x1.5mm, F.Cu at (119.6, 64.7)
- added JP22: SolderJumper_2_Bridged, Jumper:SolderJumper-2_P1.3mm_Bridged2Bar_RoundedPad1.0x1.5mm, F.Cu at (119.6, 68.2)
- added JP23: Bypass, Jumper:SolderJumper-2_P1.3mm_Open_RoundedPad1.0x1.5mm, F.Cu at (297.5, 29.5)
- added JP24: SolderJumper_2_Bridged, Jumper:SolderJumper-2_P1.3mm_Bridged2Bar_RoundedPad1.0x1.5mm, F.Cu at (297.5, 33.1)
- added JP26: SolderJumper_2_Bridged, Jumper:SolderJumper-2_P1.3mm_Bridged2Bar_RoundedPad1.0x1.5mm, F.Cu at (109.2, 84.2)
- added JP27: Bypass, Jumper:SolderJumper-2_P1.3mm_Open_RoundedPad1.0x1.5mm, F.Cu at (297.5, 49.1)
- added JP28: SolderJumper_2_Bridged, Jumper:SolderJumper-2_P1.3mm_Bridged2Bar_RoundedPad1.0x1.5mm, F.Cu at (297.5, 52.6)
- added JP3: SolderJumper_2_Bridged, Jumper:SolderJumper-2_P1.3mm_Bridged2Bar_RoundedPad1.0x1.5mm, F.Cu at (238.0, 40.6)
- added JP4: SolderJumper_2_Open, Jumper:SolderJumper-2_P1.3mm_Open_RoundedPad1.0x1.5mm, F.Cu at (269.5, -13.1)
- added JP5: SolderJumper_2_Bridged, Jumper:SolderJumper-2_P1.3mm_Bridged2Bar_RoundedPad1.0x1.5mm, F.Cu at (269.5, -9.52)
- added JP6: SolderJumper_2_Bridged, Jumper:SolderJumper-2_P1.3mm_Bridged2Bar_RoundedPad1.0x1.5mm, F.Cu at (269.5, -5.97)
- added JP7: SolderJumper_2_Open, Jumper:SolderJumper-2_P1.3mm_Open_RoundedPad1.0x1.5mm, F.Cu at (269.5, -2.42)
- added JP8: SolderJumper_2_Open, Jumper:SolderJumper-2_P1.3mm_Open_RoundedPad1.0x1.5mm, F.Cu at (238.0, 44.2)
- added JP9: SolderJumper_3_Bridged12, Jumper:SolderJumper-3_P1.3mm_Bridged12_RoundedPad1.0x1.5mm, F.Cu at (109.3, 86.8)
- added MH1 (x2): MountingHole_2.7mm_M2.5, MountingHole:MountingHole_2.7mm_M2.5, F.Cu at (382.6, 30.4)
- added MH1 (x2): MountingHole_2.7mm_M2.5, MountingHole:MountingHole_2.7mm_M2.5, F.Cu at (392.8, 115.1)
- added MH2 (x2): MountingHole_2.7mm_M2.5, MountingHole:MountingHole_2.7mm_M2.5, F.Cu at (450.8, 115.1)
- added MH2 (x2): MountingHole_2.7mm_M2.5, MountingHole:MountingHole_2.7mm_M2.5, F.Cu at (440.6, 30.4)
- added MH3: MountingHole_2.7mm_M2.5, MountingHole:MountingHole_2.7mm_M2.5, F.Cu at (382.6, 53.4)
- added MH3: MountingHole_2.7mm_M2.5, MountingHole:MountingHole_2.7mm_M2.5, F.Cu at (382.6, 79.4)
- added MH3: MountingHole_2.7mm_M2.5, MountingHole:MountingHole_2.7mm_M2.5, F.Cu at (392.8, 164.1)
- added MH3: MountingHole_2.7mm_M2.5, MountingHole:MountingHole_2.7mm_M2.5, F.Cu at (392.8, 138.1)
- added MH4: MountingHole_2.7mm_M2.5, MountingHole:MountingHole_2.7mm_M2.5, F.Cu at (440.6, 53.4)
- added MH4: MountingHole_2.7mm_M2.5, MountingHole:MountingHole_2.7mm_M2.5, F.Cu at (450.8, 164.1)
- added MH4: MountingHole_2.7mm_M2.5, MountingHole:MountingHole_2.7mm_M2.5, F.Cu at (440.6, 79.4)
- added MH4: MountingHole_2.7mm_M2.5, MountingHole:MountingHole_2.7mm_M2.5, F.Cu at (450.8, 138.1)
- added Q1: PMOS AO3401A, Package_TO_SOT_SMD:SOT-23_Handsoldering, B.Cu at (115.5, 89.5)
- added Q2: PMOS AO3401A, Package_TO_SOT_SMD:SOT-23_Handsoldering, F.Cu at (283.9, -5.67)
- added Q4: PMOS AO3401A, Package_TO_SOT_SMD:SOT-23_Handsoldering, F.Cu at (230.7, 64.3)
- added R1: 10k, Resistor_SMD:R_0603_1608Metric_Pad0.98x0.95mm_HandSolder, B.Cu at (129.1, 73.9)
- added R13: 10k, Resistor_SMD:R_0603_1608Metric_Pad0.98x0.95mm_HandSolder, B.Cu at (126.6, 73.9)
- added R14: 1k, Resistor_SMD:R_0603_1608Metric_Pad0.98x0.95mm_HandSolder, F.Cu at (265.2, -6.49)
- added R15: 1k, Resistor_SMD:R_0603_1608Metric_Pad0.98x0.95mm_HandSolder, F.Cu at (265.2, -3.98)
- added R16: 1k, Resistor_SMD:R_0603_1608Metric_Pad0.98x0.95mm_HandSolder, B.Cu at (135.7, 72.8)
- added R17: 1k, Resistor_SMD:R_0603_1608Metric_Pad0.98x0.95mm_HandSolder, B.Cu at (138.2, 72.8)
- added R18: 1k, Resistor_SMD:R_0603_1608Metric_Pad0.98x0.95mm_HandSolder, B.Cu at (140.7, 72.8)
- added R19: 10k, Resistor_SMD:R_0603_1608Metric_Pad0.98x0.95mm_HandSolder, B.Cu at (124.1, 73.9)
- added R2: 1k, Resistor_SMD:R_0603_1608Metric_Pad0.98x0.95mm_HandSolder, F.Cu at (265.2, -24.1)
- added R20: 10k, Resistor_SMD:R_0603_1608Metric_Pad0.98x0.95mm_HandSolder, B.Cu at (113.0, 90.4)
- added R21: 0, Resistor_SMD:R_0603_1608Metric_Pad0.98x0.95mm_HandSolder, F.Cu at (249.8, -2.19)
- added R22: 0, Resistor_SMD:R_0603_1608Metric_Pad0.98x0.95mm_HandSolder, F.Cu at (249.8, 0.32)
- added R23: 0, Resistor_SMD:R_0603_1608Metric_Pad0.98x0.95mm_HandSolder, F.Cu at (249.8, 2.83)
- added R24: 0, Resistor_SMD:R_0603_1608Metric_Pad0.98x0.95mm_HandSolder, F.Cu at (249.8, 5.34)
- added R25: 0, Resistor_SMD:R_0603_1608Metric_Pad0.98x0.95mm_HandSolder, F.Cu at (249.8, 7.85)
- added R26: 0, Resistor_SMD:R_0603_1608Metric_Pad0.98x0.95mm_HandSolder, F.Cu at (254.2, -2.19)
- added R27: 0, Resistor_SMD:R_0603_1608Metric_Pad0.98x0.95mm_HandSolder, F.Cu at (254.2, 0.32)
- added R28: 0, Resistor_SMD:R_0603_1608Metric_Pad0.98x0.95mm_HandSolder, F.Cu at (254.2, 2.83)
- added R29: 82k, Resistor_SMD:R_0603_1608Metric_Pad0.98x0.95mm_HandSolder, F.Cu at (293.2, 44.5)
- added R3: 10k, Resistor_SMD:R_0603_1608Metric_Pad0.98x0.95mm_HandSolder, F.Cu at (265.2, -21.6)
- added R30: 20k, Resistor_SMD:R_0603_1608Metric_Pad0.98x0.95mm_HandSolder, F.Cu at (293.2, 47.0)
- added R31: 47k, Resistor_SMD:R_0603_1608Metric_Pad0.98x0.95mm_HandSolder, F.Cu at (293.2, 49.5)
- added R32: 3.6k, Resistor_SMD:R_0603_1608Metric_Pad0.98x0.95mm_HandSolder, F.Cu at (293.2, 52.0)
- added R33: 2k, Resistor_SMD:R_0603_1608Metric_Pad0.98x0.95mm_HandSolder, F.Cu at (293.2, 54.5)
- added R34: 1k, Resistor_SMD:R_0603_1608Metric_Pad0.98x0.95mm_HandSolder, F.Cu at (293.2, 57.0)
- added R35: 10k, Resistor_SMD:R_0603_1608Metric_Pad0.98x0.95mm_HandSolder, F.Cu at (256.9, 61.1)
- added R4: 1k, Resistor_SMD:R_0603_1608Metric_Pad0.98x0.95mm_HandSolder, F.Cu at (265.2, -19.0)
- added R42: 150k, Resistor_SMD:R_0603_1608Metric_Pad0.98x0.95mm_HandSolder, F.Cu at (123.0, 57.6)
- added R43: 10k, Resistor_SMD:R_0603_1608Metric_Pad0.98x0.95mm_HandSolder, F.Cu at (123.0, 60.1)
- added R44: 47k, Resistor_SMD:R_0603_1608Metric_Pad0.98x0.95mm_HandSolder, F.Cu at (123.0, 62.6)
- added R45: 470R, Resistor_SMD:R_0603_1608Metric_Pad0.98x0.95mm_HandSolder, F.Cu at (123.0, 65.1)
- added R46: 2k, Resistor_SMD:R_0603_1608Metric_Pad0.98x0.95mm_HandSolder, F.Cu at (119.3, 53.6)
- added R47: 150k, Resistor_SMD:R_0603_1608Metric_Pad0.98x0.95mm_HandSolder, F.Cu at (293.2, 24.9)
- added R48: 10k, Resistor_SMD:R_0603_1608Metric_Pad0.98x0.95mm_HandSolder, F.Cu at (293.2, 27.4)
- added R49: 47k, Resistor_SMD:R_0603_1608Metric_Pad0.98x0.95mm_HandSolder, F.Cu at (293.2, 29.9)
- added R5: 1k, Resistor_SMD:R_0603_1608Metric_Pad0.98x0.95mm_HandSolder, F.Cu at (265.2, -16.5)
- added R50: 470R, Resistor_SMD:R_0603_1608Metric_Pad0.98x0.95mm_HandSolder, F.Cu at (293.2, 32.5)
- added R51: 2k, Resistor_SMD:R_0603_1608Metric_Pad0.98x0.95mm_HandSolder, F.Cu at (293.2, 35.0)
- added R52: 1k, Resistor_SMD:R_0603_1608Metric_Pad0.98x0.95mm_HandSolder, B.Cu at (143.2, 72.8)
- added R53: 100, Resistor_SMD:R_0603_1608Metric_Pad0.98x0.95mm_HandSolder, B.Cu at (145.7, 72.8)
- added R54: 100, Resistor_SMD:R_0603_1608Metric_Pad0.98x0.95mm_HandSolder, B.Cu at (148.2, 72.8)
- added R55: 1k, Resistor_SMD:R_0603_1608Metric_Pad0.98x0.95mm_HandSolder, B.Cu at (150.7, 72.8)
- added R56: 1k, Resistor_SMD:R_0603_1608Metric_Pad0.98x0.95mm_HandSolder, B.Cu at (135.7, 77.2)
- added R57: 1k, Resistor_SMD:R_0603_1608Metric_Pad0.98x0.95mm_HandSolder, F.Cu at (119.3, 56.1)
- added R59: 1k, Resistor_SMD:R_0603_1608Metric_Pad0.98x0.95mm_HandSolder, F.Cu at (293.2, 37.5)
- added R6: 1k, Resistor_SMD:R_0603_1608Metric_Pad0.98x0.95mm_HandSolder, F.Cu at (265.2, -14.0)
- added R60: 1k, Resistor_SMD:R_0603_1608Metric_Pad0.98x0.95mm_HandSolder, B.Cu at (138.2, 77.2)
- added R61: 100, Resistor_SMD:R_0603_1608Metric_Pad0.98x0.95mm_HandSolder, B.Cu at (140.7, 77.2)
- added R62: 1k, Resistor_SMD:R_0603_1608Metric_Pad0.98x0.95mm_HandSolder, B.Cu at (143.2, 77.2)
- added R63: 1k, Resistor_SMD:R_0603_1608Metric_Pad0.98x0.95mm_HandSolder, F.Cu at (279.6, 12.9)
- added R64: 1k, Resistor_SMD:R_0603_1608Metric_Pad0.98x0.95mm_HandSolder, F.Cu at (279.6, 15.4)
- added R65: 1k, Resistor_SMD:R_0603_1608Metric_Pad0.98x0.95mm_HandSolder, F.Cu at (279.6, 17.9)
- added R66: 1k, Resistor_SMD:R_0603_1608Metric_Pad0.98x0.95mm_HandSolder, F.Cu at (284.0, 2.85)
- added R67: 100, Resistor_SMD:R_0603_1608Metric_Pad0.98x0.95mm_HandSolder, F.Cu at (284.0, 5.36)
- added R68: 100, Resistor_SMD:R_0603_1608Metric_Pad0.98x0.95mm_HandSolder, F.Cu at (284.0, 7.87)
- added R69: 100, Resistor_SMD:R_0603_1608Metric_Pad0.98x0.95mm_HandSolder, F.Cu at (284.0, 10.4)
- added R7: 1k, Resistor_SMD:R_0603_1608Metric_Pad0.98x0.95mm_HandSolder, F.Cu at (265.2, -11.5)
- added R70: 100, Resistor_SMD:R_0603_1608Metric_Pad0.98x0.95mm_HandSolder, F.Cu at (284.0, 12.9)
- added R8: 10k, Resistor_SMD:R_0603_1608Metric_Pad0.98x0.95mm_HandSolder, F.Cu at (265.2, -9.00)
- added REF**: SolderJumper-2_P1.3mm_Open_Pad1.0x1.5mm, Jumper:SolderJumper-2_P1.3mm_Open_Pad1.0x1.5mm, F.Cu at (413.5, 150.4)
- added REF**: D_SMA, Diode_SMD:D_SMA, F.Cu at (241.4, 101.0)
- added REF**: L_Sunlord_MWSA0503S, Inductor_SMD:L_Sunlord_MWSA0503S, F.Cu at (217.4, 61.8)
- added REF**: D_SOD-323, Diode_SMD:D_SOD-323, F.Cu at (241.0, 92.8)
- added REF**: D_SOD-123, Diode_SMD:D_SOD-123, F.Cu at (241.0, 96.6)
- added REF**: Pololu_Breakout-16_15.2x20.3mm, Module:Pololu_Breakout-16_15.2x20.3mm, F.Cu at (431.8, 156.3)
- added REF**: SOIC-8-1EP_3.9x4.9mm_P1.27mm_EP2.29x3mm, Package_SO:SOIC-8-1EP_3.9x4.9mm_P1.27mm_EP2.29x3mm, F.Cu at (210.0, 61.6)
- added REF**: SOIC-8-1EP_3.9x4.9mm_P1.27mm_EP2.29x3mm, Package_SO:SOIC-8-1EP_3.9x4.9mm_P1.27mm_EP2.29x3mm, F.Cu at (210.2, 67.8)
- added REF**: C_0603_1608Metric, Capacitor_SMD:C_0603_1608Metric, F.Cu at (245.6, 95.2)
- added REF**: D_SOD-323_HandSoldering, Diode_SMD:D_SOD-323_HandSoldering, F.Cu at (241.0, 91.0)
- added REF**: SolderJumper-2_P1.3mm_Open_Pad1.0x1.5mm, Jumper:SolderJumper-2_P1.3mm_Open_Pad1.0x1.5mm, F.Cu at (413.5, 148.4)
- added REF**: SolderJumper-2_P1.3mm_Open_Pad1.0x1.5mm, Jumper:SolderJumper-2_P1.3mm_Open_Pad1.0x1.5mm, F.Cu at (413.5, 146.4)
- added REF**: L_Sunlord_MWSA0503S, Inductor_SMD:L_Sunlord_MWSA0503S, F.Cu at (217.6, 67.6)
- added REF**: Pololu_Breakout-16_15.2x20.3mm, Module:Pololu_Breakout-16_15.2x20.3mm, F.Cu at (411.5, 156.3)
- added SW1: SW_Push TODO FP CHECK, Button_Switch_SMD:SW_SPST_SKQG_WithStem, F.Cu at (241.0, 80.0)
- added TP1: TestPoint, Connector_PinSocket_2.54mm:PinSocket_1x01_P2.54mm_Vertical, F.Cu at (258.4, 37.6)
- added TP2: TestPoint, Connector_PinSocket_2.54mm:PinSocket_1x01_P2.54mm_Vertical, F.Cu at (258.4, 42.2)
- added TP3: TestPoint, Connector_PinSocket_2.54mm:PinSocket_1x01_P2.54mm_Vertical, F.Cu at (258.4, 46.8)
- added TP4: TestPoint, Connector_PinSocket_2.54mm:PinSocket_1x01_P2.54mm_Vertical, F.Cu at (250.0, 19.1)
- added TP5: TestPoint, Connector_PinSocket_2.54mm:PinSocket_1x01_P2.54mm_Vertical, F.Cu at (274.0, -12.5)
- added TP6: TestPoint, Connector_PinSocket_2.54mm:PinSocket_1x01_P2.54mm_Vertical, F.Cu at (274.0, -7.92)
- added TP7: TestPoint, Connector_PinSocket_2.54mm:PinSocket_1x01_P2.54mm_Vertical, F.Cu at (274.0, -3.32)
- added U2: TPS25963x, Package_SO:SOIC-8-1EP_3.9x4.9mm_P1.27mm_EP2.95x4.9mm_Mask2.71x3.4mm_ThermalVias, B.Cu at (147.1, 56.1)
- added U3: AMS1117-3.3, Package_TO_SOT_SMD:SOT-223-3_TabPin2, B.Cu at (87.2, 83.2)
- added U4: CH224K, 0chessbot-parts:SSOP-10-1EP_3.9x4.9mm_P1mm_EP2.1x3.3mm, B.Cu at (113.4, 57.6)
- added U5: TPS25963x, Package_SO:SOIC-8-1EP_3.9x4.9mm_P1.27mm_EP2.95x4.9mm_Mask2.71x3.4mm_ThermalVias, F.Cu at (299.6, 24.5)
- added U6: TPS25963x, Package_SO:SOIC-8-1EP_3.9x4.9mm_P1.27mm_EP2.95x4.9mm_Mask2.71x3.4mm_ThermalVias, F.Cu at (299.6, 44.1)
- moved J?? 376.9 mm to (396.5, -30.4)
- moved MH1 376.9 mm to (391.7, -31.7)
- moved MH2 376.9 mm to (449.7, -31.7)
- moved MH3 376.9 mm to (391.7, -8.67)
- moved MH4 376.9 mm to (449.7, -8.67)
- moved REF** 297.2 mm to (413.4, 152.4)
- moved REF** 297.2 mm to (396.2, 151.4)
- moved REF** 297.2 mm to (392.9, 124.8)
- moved REF** 297.2 mm to (397.5, 162.5)
- moved REF** 297.2 mm to (421.8, 115.1)
- renumbered J1 to J??
Other:
- board size 319.5 x 172 mm -> 354.4 x 202.8 mm

Commit message: pcb layout work
Parts:
- removed D22: G, LED_SMD:LED_0603_1608Metric_Pad1.05x0.95mm_HandSolder
- removed J8: Conn_01x02_Pin, Connector_PinHeader_2.54mm:PinHeader_1x02_P2.54mm_Vertical
- removed J?? (x5): GPIO, Connector_PinSocket_2.54mm:PinSocket_2x20_P2.54mm_Vertical
- removed the MH1 at (103.4, 47.5) (x2)
- removed the MH2 at (161.4, 47.5) (x2)
- removed Q4: PMOS AO3401A, Package_TO_SOT_SMD:SOT-23_Handsoldering
- removed R21, R22, R23, R24, R25, R26, R27, R28: 0, Resistor_SMD:R_0603_1608Metric_Pad0.98x0.95mm_HandSolder
- removed R35: 10k, Resistor_SMD:R_0603_1608Metric_Pad0.98x0.95mm_HandSolder
- removed REF**: PinSocket_2x20_P2.54mm_Horizontal, Connector_PinSocket_2.54mm:PinSocket_2x20_P2.54mm_Horizontal
- removed REF** (x3): SolderJumper-2_P1.3mm_Open_Pad1.0x1.5mm, Jumper:SolderJumper-2_P1.3mm_Open_Pad1.0x1.5mm
- removed REF**: D_SMA, Diode_SMD:D_SMA
- removed REF** (x2): L_Sunlord_MWSA0503S, Inductor_SMD:L_Sunlord_MWSA0503S
- removed REF**: D_SOD-323, Diode_SMD:D_SOD-323
- removed REF**: R_0603_1608Metric_Pad0.98x0.95mm_HandSolder, Resistor_SMD:R_0603_1608Metric_Pad0.98x0.95mm_HandSolder
- removed REF**: BarrelJack_CUI_PJ-063AH_Horizontal, Connector_BarrelJack:BarrelJack_CUI_PJ-063AH_Horizontal
- removed REF**: D_SOD-123, Diode_SMD:D_SOD-123
- removed REF**: USB_C_Receptacle_GCT_USB4105-xx-A_16P_TopMnt_Horizontal, Connector_USB:USB_C_Receptacle_GCT_USB4105-xx-A_16P_TopMnt_Horizontal
- removed REF** (x2): Pololu_Breakout-16_15.2x20.3mm, Module:Pololu_Breakout-16_15.2x20.3mm
- removed REF** (x2): SOIC-8-1EP_3.9x4.9mm_P1.27mm_EP2.29x3mm, Package_SO:SOIC-8-1EP_3.9x4.9mm_P1.27mm_EP2.29x3mm
- removed REF**: C_0603_1608Metric, Capacitor_SMD:C_0603_1608Metric
- removed REF**: D_SOD-323_HandSoldering, Diode_SMD:D_SOD-323_HandSoldering
- removed REF**: PinSocket_2x20_P2.54mm_Vertical_SMD, Connector_PinSocket_2.54mm:PinSocket_2x20_P2.54mm_Vertical_SMD
- removed SW1: SW_Push TODO FP CHECK, Button_Switch_SMD:SW_SPST_SKQG_WithStem
- removed TP2: TestPoint, Connector_PinSocket_2.54mm:PinSocket_1x01_P2.54mm_Vertical
- added JP25: SolderJumper_2_Bridged, Jumper:SolderJumper-2_P1.3mm_Bridged2Bar_RoundedPad1.0x1.5mm, F.Cu at (118.8, 53.9)
- added JP29: SolderJumper_2_Open, Jumper:SolderJumper-2_P1.3mm_Open_RoundedPad1.0x1.5mm, F.Cu at (144.4, 72.0)
- added JP30: SolderJumper_2_Open, Jumper:SolderJumper-2_P1.3mm_Open_RoundedPad1.0x1.5mm, F.Cu at (129.5, 71.9)
- added JTMP??: GPIO, Connector_PinSocket_2.54mm:PinSocket_2x20_P2.54mm_Vertical, B.Cu at (108.4, 48.8)
- added MH1: MountingHole_2.7mm_M2.5, MountingHole:MountingHole_2.7mm_M2.5, F.Cu at (103.5, 47.5)
- added MH2: MountingHole_2.7mm_M2.5, MountingHole:MountingHole_2.7mm_M2.5, F.Cu at (161.5, 47.5)
- added SW2: SW_Push TODO FP CHECK, Button_Switch_SMD:SW_SPST_SKQG_WithStem, F.Cu at (170.3, -1.90)
- added TP10: TestPoint, TestPoint:TestPoint_THTPad_1.0x1.0mm_Drill0.5mm, F.Cu at (133.7, 71.7)
- added TP11: TestPoint, TestPoint:TestPoint_THTPad_1.0x1.0mm_Drill0.5mm, F.Cu at (108.6, 64.4)
- added TP12: TestPoint, TestPoint:TestPoint_THTPad_1.0x1.0mm_Drill0.5mm, F.Cu at (108.6, 61.2)
- added TP13: TestPoint, TestPoint:TestPoint_THTPad_1.0x1.0mm_Drill0.5mm, F.Cu at (108.8, 56.6)
- added TP14: TestPoint, TestPoint:TestPoint_THTPad_1.0x1.0mm_Drill0.5mm, F.Cu at (116.0, 61.8)
- added TP15: TestPoint, Connector_PinSocket_2.54mm:PinSocket_1x01_P2.54mm_Vertical, F.Cu at (167.8, 3.80)
- added TP8: TestPoint, TestPoint:TestPoint_THTPad_1.0x1.0mm_Drill0.5mm, F.Cu at (141.1, 71.7)
- added TP9: TestPoint, TestPoint:TestPoint_THTPad_1.0x1.0mm_Drill0.5mm, F.Cu at (148.6, 71.8)
- C11, C13, C2, C5, C6, C7, C8, D11, D12, D13, D26, D27, D28, D29, D30, JP21, JP22, JP23, JP24, JP27, JP28, Q2, R14, R15, R2, R29, R3, R30, R31, R32, R33, R34, R4, R42, R43, R44, R45, R46, R47, R48, R49, R5, R50, R51, R57, R59, R6, R67, R7, R8, TP4: moved to B.Cu
- D4: value G -> Y; moved to B.Cu
- J27: footprint Connector_PinSocket_2.54mm:PinSocket_2x20_P2.54mm_Vertical_SMD -> Connector_Samtec_HLE_SMD:Samtec_HLE-120-02-xxx-DV-BE-A_2x20_P2.54mm_Horizontal; moved to B.Cu
- JP13, JP14, JP15, JP16, JP17: footprint TestPoint:TestPoint_2Pads_Pitch2.54mm_Drill0.8mm -> 0chessbot-parts:Bridged_TestPoint_2Pads_Pitch2.54mm_Drill0.8mm
- U2: footprint Package_SO:SOIC-8-1EP_3.9x4.9mm_P1.27mm_EP2.95x4.9mm_Mask2.71x3.4mm_ThermalVias -> Package_SO:TI_SO-PowerPAD-8
- U5, U6: footprint Package_SO:SOIC-8-1EP_3.9x4.9mm_P1.27mm_EP2.95x4.9mm_Mask2.71x3.4mm_ThermalVias -> Package_SO:TI_SO-PowerPAD-8; moved to B.Cu
- moved C9 223.1 mm to (2.50, 1.18)
- moved D29 205.7 mm to (105.3, 78.7), turned to 180 degrees
- moved D30 189.1 mm to (123.5, 57.2), turned to 90 degrees
- moved Q2 177.8 mm to (116.0, 52.8), turned to 180 degrees
- moved D32 173.8 mm to (129.6, 73.9)
- moved R67 172.8 mm to (138.8, 99.0), turned to 180 degrees
- moved R7 171.9 mm to (110.9, 64.4), turned to 90 degrees
- moved D31 170.8 mm to (133.0, 73.9)
- moved U6 170.0 mm to (130.6, 63.0), turned to -90 degrees
- moved JP4 167.7 mm to (115.4, 53.1)
- moved R5 166.9 mm to (117.0, 60.2)
- moved R4 166.6 mm to (117.0, 57.0)
- moved R8 166.3 mm to (111.2, 53.8), turned to 180 degrees
- moved JP27 165.5 mm to (133.2, 68.8)
- moved JP6 165.1 mm to (118.8, 61.4)
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Connections:
- net /ChessBoard/RESERVED renamed Net-(J3-Pin_5)
- net /GPIO10/SPI0.MOSI renamed /LCD/TP_SI
- net /GPIO11/SPI0.SCLK renamed /LED/TP_SCK
- net /GPIO12/PWM0 renamed /LED_DATA
- net /GPIO13/PWM1 renamed Net-(J27-Pin_33)
- net /GPIO14/TXD0 renamed Net-(J27-Pin_8)
- net /GPIO15/RXD0 renamed Net-(J27-Pin_10)
- net /GPIO16 renamed Net-(J27-Pin_36)
- net /GPIO17 renamed /TP_IRQ
- net /GPIO18/PCM.CLK renamed Net-(J27-Pin_12)
- net /GPIO19/PCM.FS renamed Net-(J27-Pin_35)
- net /GPIO20/PCM.DIN renamed Net-(J27-Pin_38)
- net /GPIO21/PCM.DOUT renamed Net-(J27-Pin_40)
- net /GPIO22 renamed Net-(J27-Pin_15)
- net /GPIO23 renamed Net-(J27-Pin_16)
- net /GPIO24 renamed /LCD_RS
- net /GPIO25 renamed /LCD_RST
- net /GPIO26 renamed Net-(J27-Pin_37)
- net /GPIO27 renamed Net-(J27-Pin_13)
- net /GPIO2/SDA1 renamed Net-(J27-Pin_3)
- net /GPIO3/SCL1 renamed Net-(J27-Pin_5)
- net /GPIO4/GPCLK0 renamed Net-(J27-Pin_7)
- net /GPIO5 renamed Net-(J27-Pin_29)
- net /GPIO6 renamed Net-(J27-Pin_31)
- net /GPIO7/SPI0.CE1 renamed /TP_CS
- net /GPIO8/SPI0.CE0 renamed /LCD_CS
- net /GPIO9/SPI0.MISO renamed /TP_SO
- C4 pad 1: /CH_3V3 -> /ChessBoard/3V3
- D10 pad 2: /Power/CNC_VIO -> /PI_3V3
- D11 pad 1: Net-(D11-K) -> GND
- D12 pad 1: Net-(D12-K) -> /DIR1
- D13 pad 1: Net-(D13-K) -> GND
- D15 pad 2: /LED_IN -> /ChessBoard/LED_IN
- D26 pad 1: Net-(D26-K) -> GND
- D27 pad 1: Net-(D27-K) -> GND
- D28 pad 1: Net-(D28-K) -> /DIR2
- D4 pad 1: Net-(D4-K) -> /ENBL
- J11 pad 1: /Power/EN -> unconnected-(J11-Pin_1-Pad1)
- J2 pad 1: (no net) -> /LIM_SW1
- J2 pad 2: (no net) -> GND
- J2 pad 3: (no net) -> /LIM_SW2
- J2 pad 4: (no net) -> GND
- J2 pad 5: (no net) -> /LIM_SW3
- J2 pad 6: (no net) -> GND
- J2 pad 7: (no net) -> /LIM_SW4
- J2 pad 8: (no net) -> GND
- J5 pad 1: (no net) -> /MAG_PWM
- J5 pad 2: (no net) -> /CNC/VIO
- J5 pad 3: (no net) -> Net-(J5-Pin_3)
- J5 pad 4: (no net) -> /CNC/SERVO_VIN
- J5 pad 5: (no net) -> GND
- J5 pad 6: (no net) -> GND
- J5 pad 7: (no net) -> GND
- J5 pad 8: (no net) -> Net-(D1-K)
- J6 pad 1: GND -> /Power/PWR_SW_B
- J6 pad 2: /ID_SCL -> GND
- J6 pad 3: /ID_SDA -> /ID_SCL
- J6 pad 4: /LED_IN -> /ID_SDA
- J6 pad 8: /CH_3V3 -> /Power/PWR_SW_A
- JP1 pad 2: /CH_3V3 -> /ChessBoard/3V3
- JP19 pad 1: /CH_5V -> GND
- JP19 pad 2: /CH_5V -> Net-(JP19-B)
- JP2 pad 2: Net-(J5-Pin_a2) -> Net-(J5-Pin_3)
- JP20 pad 2: /Power/UNLIM_5V -> /CH_5V
- JP8 pad 1: /LED_IN -> /ChessBoard/LED_IN
- Q2 pad 2: Net-(Q2-G) -> /Power/PWR_SW_B
- R3 pad 2: Net-(Q2-G) -> /Power/PWR_SW_B
- R42 pad 2: Net-(U2-EN/UVLO) -> Net-(JP19-B)
- R43 pad 1: Net-(U2-EN/UVLO) -> Net-(JP19-B)
- TP4 pad 1: /CNC/VIO -> /CNC/VMOT
- TP7 pad 1: /Power/CNC_VIO -> /PI_3V3
- U2 pad 3: Net-(U2-EN/UVLO) -> Net-(JP19-B)
- U3 pad 2: /CH_3V3 -> /ChessBoard/3V3
- U4 pad 10: Net-(Q2-G) -> /Power/PWR_SW_A
- U4 pad 11: (no net) -> GND
Routing:
- net /Power/UNLIM_5V: track 0.00 -> 52.7 mm
- net GND: track 0.00 -> 39.0 mm, vias 0 -> 15
- net Net-(JP4-A): track 0.00 -> 38.3 mm, vias 0 -> 3
- net Net-(D21-A): track 0.00 -> 33.8 mm, vias 0 -> 1
- net Net-(D20-A): track 0.00 -> 33.8 mm, vias 0 -> 1
- net Net-(D31-A): track 0.00 -> 33.8 mm, vias 0 -> 1
- net /Power/UNLIM_VIN: track 0.00 -> 29.4 mm
- net Net-(JP30-B): track 0.00 -> 23.7 mm, vias 0 -> 1
- net Net-(JP29-B): track 0.00 -> 23.7 mm, vias 0 -> 1
- net Net-(JP19-B): track 0.00 -> 23.7 mm, vias 0 -> 1
- net /PI_3V3: track 0.00 -> 21.8 mm
- net /Power/CH_VDD: track 0.00 -> 15.2 mm, vias 0 -> 1
- net Net-(JP7-B): track 0.00 -> 12.0 mm
- net Net-(D30-A): track 0.00 -> 11.1 mm, vias 0 -> 1
- net /Power/CNC_VIO: track 0.00 -> 10.7 mm
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- added copper zone on B.Cu, net GND
- added copper zone on F.Cu, net GND
Other:
- board size 354.4 x 202.8 mm -> 65 x 53 mm

Commit message: progress
Parts:
- removed JP25, JP3: SolderJumper_2_Bridged, Jumper:SolderJumper-2_P1.3mm_Bridged2Bar_RoundedPad1.0x1.5mm
- removed JTMP??: GPIO, Connector_PinSocket_2.54mm:PinSocket_2x20_P2.54mm_Vertical
- added C15: 100u, Capacitor_SMD:CP_Elec_6.3x5.4, F.Cu at (149.8, 84.4)
- added D9: 20V+ D_TVS, Diode_SMD:D_SOD-123F, B.Cu at (140.9, 87.7)
- added R10: 1k, Resistor_SMD:R_0603_1608Metric_Pad0.98x0.95mm_HandSolder, B.Cu at (113.2, 90.8)
- added R11: 1k, Resistor_SMD:R_0603_1608Metric_Pad0.98x0.95mm_HandSolder, F.Cu at (160.8, 51.6)
- added R12: 1k, Resistor_SMD:R_0603_1608Metric_Pad0.98x0.95mm_HandSolder, B.Cu at (159.9, 64.3)
- added R21: 1k, Resistor_SMD:R_0603_1608Metric_Pad0.98x0.95mm_HandSolder, B.Cu at (136.9, 98.9)
- added R9: 1k, Resistor_SMD:R_0603_1608Metric_Pad0.98x0.95mm_HandSolder, B.Cu at (110.8, 90.8)
- C1: value 100u -> 22uF; footprint Capacitor_SMD:CP_Elec_6.3x5.4 -> Capacitor_SMD:C_1206_3216Metric_Pad1.33x1.80mm_HandSolder; moved to B.Cu
- C12, C14, C3, C4, C9, D1, D16, D17, D18, D5, D8, JP18, JP8, R63, R64, R65, R66, R68, R69, R70: moved to B.Cu
- D11, D12, D13, D26, D27, D28, D4: moved to F.Cu
- TP1, TP3: footprint Connector_PinSocket_2.54mm:PinSocket_1x01_P2.54mm_Vertical -> Connector_PinHeader_1.00mm:PinHeader_1x01_P1.00mm_Vertical
- TP6: footprint Connector_PinSocket_2.54mm:PinSocket_1x01_P2.54mm_Vertical -> TestPoint:TestPoint_THTPad_1.5x1.5mm_Drill0.7mm
- moved D2 150.5 mm to (101.3, 75.0), turned to 90 degrees
- moved D10 148.3 mm to (102.0, 53.7)
- moved R70 142.9 mm to (113.5, 86.9), turned to 90 degrees
- moved R69 141.6 mm to (115.0, 86.9), turned to -90 degrees
- moved TP7 140.8 mm to (105.1, 51.4)
- moved C9 139.9 mm to (124.9, 68.9), turned to 90 degrees
- moved TP5 137.2 mm to (110.9, 73.2)
- moved C7 128.0 mm to (106.3, 54.4), turned to 180 degrees
- moved R66 128.0 mm to (130.0, 87.2), turned to 90 degrees
- moved C12 127.4 mm to (126.4, 60.5), turned to -90 degrees
- moved R65 126.2 mm to (125.1, 80.3), turned to -90 degrees
- moved TP1 125.6 mm to (148.8, 98.9), turned to 180 degrees
- moved JP8 124.8 mm to (116.3, 71.4), turned to -90 degrees
- moved JP18 124.5 mm to (115.9, 79.1), turned to 180 degrees
- moved R63 123.9 mm to (127.7, 80.3), turned to -90 degrees
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Connections:
- D6 pad 2: /ChessBoard/LED_OUT -> Net-(D6-DOUT)
- J1 pad 1: Net-(A2-1B) -> Net-(A1-1B)
- J1 pad 2: Net-(A2-1A) -> Net-(A2-1B)
- J1 pad 3: Net-(A2-2A) -> Net-(A1-1A)
- J1 pad 4: Net-(A2-2B) -> Net-(A2-1A)
- J1 pad 5: Net-(A1-1B) -> Net-(A1-2A)
- J1 pad 6: Net-(A1-1A) -> Net-(A2-2A)
- J1 pad 7: Net-(A1-2A) -> Net-(A1-2B)
- J1 pad 8: Net-(A1-2B) -> Net-(A2-2B)
- J27 pad 32: /LED_DATA -> Net-(J27-Pin_32)
- J3 pad 2: /CH_SDA -> /ChessBoard/LED_OUT
- J3 pad 3: /CH_SCL -> /CH_SDA
- J3 pad 5: Net-(J3-Pin_5) -> /CH_SCL
- J3 pad 8: /ChessBoard/LED_OUT -> Net-(J3-Pin_8)
- J6 pad 2: GND -> /Power/PWR_SW_A
- J6 pad 3: /ID_SCL -> /ID_SDA
- J6 pad 4: /ID_SDA -> /CH_5V
- J6 pad 5: /Power/UNLIM_VIN -> /ID_SCL
- J6 pad 6: /PI_5V -> GND
- J6 pad 7: /CH_5V -> unconnected-(J6-Pin_7-Pad7)
- J6 pad 8: /Power/PWR_SW_A -> /Power/UNLIM_VIN
- JP1 pad 1: Net-(J3-Pin_4) -> Net-(J3-Pin_7)
- JP12 pad 1: /ChessBoard/LED_OUT -> Net-(D6-DOUT)
- R16 pad 2: /DIR1 -> /LIM_SW2
- R17 pad 2: /STEP1 -> /LIM_SW3
- R63 pad 1: /LIM_SW1 -> /STEP1
- R64 pad 1: /LIM_SW2 -> /LIM_SW4
- R65 pad 1: Net-(J27-Pin_16) -> /DIR1
- R65 pad 2: /LIM_SW3 -> Net-(J27-Pin_16)
- R66 pad 1: /LIM_SW4 -> /LIM_SW1
- R69 pad 2: /ID_SCL -> Net-(R10-Pad1)
- R70 pad 1: /ID_SDA -> Net-(R70-Pad1)
- TP1 pad 1: Net-(J3-Pin_5) -> Net-(J3-Pin_8)
- TP3 pad 1: Net-(J3-Pin_5) -> Net-(J3-Pin_8)
Routing:
- net GND: track 39.0 -> 154.8 mm, vias 15 -> 42
- net /CNC/VIO: track 0.00 -> 103.7 mm, vias 0 -> 5
- net Net-(J27-Pin_33): track 0.00 -> 67.8 mm, vias 0 -> 2
- net Net-(J27-Pin_3): track 1.22 -> 65.8 mm, vias 1 -> 2
- net Net-(J27-Pin_27): track 0.00 -> 64.0 mm, vias 0 -> 2
- net Net-(J27-Pin_28): track 0.00 -> 61.9 mm, vias 0 -> 2
- net Net-(J27-Pin_5): track 1.40 -> 61.9 mm, vias 1 -> 2
- net Net-(J27-Pin_8): track 0.00 -> 54.4 mm
- net Net-(J27-Pin_10): track 0.00 -> 53.9 mm
- net Net-(J27-Pin_15): track 0.00 -> 47.9 mm, vias 0 -> 2
- net Net-(J27-Pin_12): track 0.00 -> 47.5 mm, vias 0 -> 2
- net /Power/UNLIM_VIN: track 29.4 -> 76.4 mm
- net /ChessBoard/LED_OUT: track 0.00 -> 46.6 mm
- net /Power/PWR_SW_A: track 4.75 -> 51.2 mm, vias 1 -> 2
- net Net-(J27-Pin_7): track 0.00 -> 46.2 mm
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- added copper zone on In1.Cu, net /PI_5V
- added copper zone on In2.Cu, net GND
- removed copper zone on B.Cu, net GND
- removed copper zone on F.Cu, net GND
Other:
- board size 65 x 53 mm -> 65 x 56.5 mm
- copper layers 2 -> 4
- board text added: "TBD Remove"

Commit message: yay its all connected
Parts:
- removed the MH1 at (382.6, 30.4) (x2)
- removed the MH1 at (392.8, 115.1) (x2)
- removed the MH1 at (391.7, -31.7)
- removed the MH2 at (450.8, 115.1) (x2)
- removed the MH2 at (440.6, 30.4) (x2)
- removed the MH2 at (449.7, -31.7)
- removed the MH3 at (391.7, -8.67)
- removed the MH3 at (382.6, 53.4)
- removed the MH3 at (382.6, 79.4)
- removed the MH3 at (392.8, 164.1)
- removed the MH3 at (392.8, 138.1)
- removed the MH4 at (440.6, 53.4)
- removed the MH4 at (450.8, 164.1)
- removed the MH4 at (440.6, 79.4)
- removed the MH4 at (449.7, -8.67)
- removed the MH4 at (450.8, 138.1)
- TP1, TP3: footprint Connector_PinHeader_1.00mm:PinHeader_1x01_P1.00mm_Vertical -> TestPoint:TestPoint_THTPad_1.0x1.0mm_Drill0.5mm
- TP15, TP4, TP5, TP7: footprint Connector_PinSocket_2.54mm:PinSocket_1x01_P2.54mm_Vertical -> TestPoint:TestPoint_THTPad_D2.0mm_Drill1.0mm
- moved JP10 11.7 mm to (110.2, 78.9)
Connections:
- J27 pad 1: /PI_3V3 -> unconnected-(J27-Pin_1-Pad1)
Routing:
- net /CH_5V: track 28.0 -> 138.5 mm, vias 0 -> 10
- net /CNC/VMOT: track 19.5 -> 99.9 mm, vias 0 -> 4
- net /Power/UNLIM_VIN: track 76.4 -> 118.4 mm
- net Net-(JP9-C): track 5.33 -> 11.1 mm
- net GND: track 154.8 -> 151.4 mm
- net Net-(J27-Pin_36): track 42.0 -> 42.7 mm
- net Net-(J27-Pin_38): track 42.0 -> 41.6 mm, vias 0 -> 2
- added copper zone on In1.Cu, net /CH_5V
Other:
- outline, holes or cut-outs redrawn
- board text removed: "4mm clearance (incl.)"
- board text removed: "5mm clearance (incl.)"
- board text removed: "6mm clearance (incl. 1 safety)"
- board text removed: "CAMERA (OPTIONAL)"
- board text removed: "DISPLAY (OPTIONAL)"
- board text removed: "Extend PCB edge 0.5mm if using SMT header"
- board text removed: "SD Card clearance"

Commit message: a
Parts:
- A1, A2: footprint Module:Pololu_Breakout-16_15.2x20.3mm -> 0chessbot-parts:Pololu_Breakout-16_15.2x20.3mm
- J27: footprint Connector_Samtec_HLE_SMD:Samtec_HLE-120-02-xxx-DV-BE-A_2x20_P2.54mm_Horizontal -> 0chessbot-parts:Samtec_HLE-120-02-xxx-DV-BE-A_2x20_P2.54mm_Horizontal
- J4: footprint Connector_USB:USB_C_Receptacle_HRO_TYPE-C-31-M-12 -> 0chessbot-parts:USB_C_Receptacle_HRO_TYPE-C-31-M-12
- J7: footprint TerminalBlock_RND:TerminalBlock_RND_205-00287_1x02_P5.08mm_Horizontal -> TerminalBlock_Phoenix:TerminalBlock_Phoenix_PT-1,5-2-5.0-H_1x02_P5.00mm_Horizontal
- Q1, Q2: footprint Package_TO_SOT_SMD:SOT-23_Handsoldering -> Package_TO_SOT_SMD:SOT-23
- SW2: footprint Button_Switch_SMD:SW_SPST_SKQG_WithStem -> 0chessbot-parts:SW_SPST_SKQG_WithStem
- moved J7 4.84 mm to (102.8, 83.9), turned to -90 degrees
- moved TP4 1.14 mm to (162.7, 92.5)
Connections:
- J7 pad 1: GND -> Net-(D29-A)
- J7 pad 2: Net-(D29-A) -> GND
Routing:
- net GND: track 151.4 -> 156.0 mm
- net /Power/UNLIM_5V: track 62.7 -> 59.3 mm
- net /CNC/VIO: track 103.7 -> 104.4 mm
