File: controlboard/controlboard.kicad_pcb (KiCad board)
At the start: 4 copper layers, 65 x 56.5 mm, 167 parts, among them J1 Conn_02x04_Counter_Clockwise, J11 Pololu Voltage Regulator, J2 Conn_02x04_Row_Letter_Last, J27 GPIO, J3 Conn_02x04_Counter_Clockwise, J4 USB_C_Receptacle_USB2.0_14P, J5 Conn_02x04_Row_Letter_First, J6 Conn_02x04_Counter_Clockwise, J7 Screw_Terminal_01x02, J9 mini560 voltage regulator, Q1 NMOS AO3400A, Q2 PMOS AO3401A, SW2 SW_Push TODO FP CHECK, U2 TPS25963x, U3 AMS1117-3.3, U4 CH224K, U5 TPS25963x, U6 TPS25963x

Commit message: improvements
Parts:
- removed D16: 20V+ D_TVS, Diode_SMD:D_SOD-123F
- R32: value 3.6k -> 3k
- R33, R46, R51: value 2k -> 3k
- moved TP6 0.80 mm to (157.9, 59.5)
- moved D3 0.51 mm to (155.9, 59.5)
Routing:
- net GND: track 149.1 -> 136.7 mm, vias 43 -> 35
- net Net-(D7-VDD): track 3.40 -> 4.46 mm
- net /CH_5V: track 138.2 -> 139.0 mm
- net Net-(J27-Pin_32): track 18.7 -> 19.5 mm, vias 1 -> 2
- net /PI_5V: vias 6 -> 3
Other:
- board text added: "5V"
- board text added: "CC1"
- board text added: "CC2"
- board text added: "JLCJLCJLCJLC"
- board text added: "PI_3V3"

Commit message: nice silkscreen stuff
Parts:
- added G***: LOGO, LOGO, F.Cu at (139.9, 65.8)
- J4: value USB_C_Receptacle_USB2.0_14P -> TYPE-C-31-M-12
- R11: moved to B.Cu
- moved R11 3.23 mm to (158.3, 53.7)
Routing:
- net Net-(J27-Pin_32): track 19.5 -> 22.8 mm
- net /LED_DATA: track 6.05 -> 7.51 mm, vias 0 -> 1
Other:
- board text added: "Designed by Karmanyaah Malhotra June 2024"
- board text added: "Hi future RASers! Email me at karmanyaah@malhotra.cc if you see"
- board text added: "UT IEEE RAS ChessBot ControlBoard June '24"
- board text added: "https://github.com/ut-ras/chessbot"
- board text added: "https://k.malhotra.cc"
- board text added: "this!!"

Commit message: update pcb easter egg
Other:
- board text added: "Hi future RAScals! Email me at karras@malhotra.cc if you see this!!"
- board text removed: "Hi future RASers! Email me at karmanyaah@malhotra.cc if you see"
- board text removed: "this!!"
Changed lines of the file:
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@@
 		)
 	)
-	(gr_text "this!!"
-		(at 106.858 50.096 0)
-		(layer "B.SilkS")
-		(effects
-			(font
-				(size 1 0.9)
-				(thickness 0.15)
-				(bold yes)
-			)
-			(justify left bottom mirror)
-		)
-	)
-	(gr_text "Hi future RASers! Email me at karmanyaah@malhotra.cc if you   see"
+	(gr_text "Hi future RAScals! Email me at karras@malhotra.cc if you see    this!!"
 		(at 154.102 48.064 0)
 		(layer "B.SilkS")

Commit message: controlboard finalized and ordered!!!
Parts:
- added REF**: MountingHole_2.1mm, MountingHole:MountingHole_2.1mm, F.Cu at (101.7, 50.8)
- added REF**: MountingHole_2.1mm, MountingHole:MountingHole_2.1mm, F.Cu at (163.3, 87.7)
- added REF**: MountingHole_2.1mm, MountingHole:MountingHole_2.1mm, F.Cu at (163.0, 49.9)
- moved C7 0.21 mm to (106.3, 54.2)
Routing:
- net GND: track 136.7 -> 131.4 mm
- net /CNC/VMOT: track 158.8 -> 155.2 mm
- net /Power/VBUS: track 70.1 -> 66.7 mm
- net /LED_DATA: track 7.51 -> 4.39 mm
- net /Power/UNLIM_5V: track 59.3 -> 56.5 mm
- net Net-(U4-CFG1): track 7.88 -> 6.17 mm, vias 1 -> 0
- net /CH_5V: track 139.0 -> 137.6 mm
- net /CNC/VIO: track 104.4 -> 103.2 mm
- net Net-(D30-A): track 11.2 -> 10.1 mm
- net Net-(J27-Pin_32): track 22.8 -> 23.7 mm
- net Net-(Q2-G): track 19.6 -> 18.7 mm
- net /Power/PWR_SW_A: track 51.2 -> 50.6 mm
- net /ChessBoard/LED_IN: track 8.74 -> 8.20 mm
- net Net-(J27-Pin_28): track 61.9 -> 61.5 mm, vias 2 -> 3
Other:
- board size 65 x 56.5 mm -> 65 x 57 mm
- board text added: "+"
- board text added: "GND"
