File: chessboard5/cell.kicad_sch (KiCad schematic)
At the start: 9 parts, among them Q1 AO3401A, U1 WS2814F, U2 TMAG5273

Commit message: Progress!!!
Connections:
- net GND: now also C2.2
- net +3V3 renamed +3.3V
- net 5V renamed +5V

Commit message: finished chessboard v5!!!
Parts:
- U5: renamed from U1; footprint Package_TO_SOT_SMD:SOT-23-8_Handsoldering -> 0chessbot:FSOP-8
- renumbered C1 to C7, C2 to C8, C3 to C9, D1 to D3, Q1 to Q3, R1 to R5, R2 to R6, U2 to U6
Changed lines of the file:
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@@
 	(paper "A4")
+	(junction
+		(at 189.23 74.93)
+		(diameter 0)
+		(color 0 0 0 0)
+	)
 	(junction
 		(at 139.7 69.85)
@@
 		(color 0 0 0 0)
 	)
+	(junction
+		(at 96.52 82.55)
+		(diameter 0)
+		(color 0 0 0 0)
+	)
 	(wire
 		(pts
@@
 	(wire
 		(pts
-			(xy 96.52 81.28) (xy 96.52 83.82)
+			(xy 96.52 81.28) (xy 96.52 82.55)
 		)
 		(stroke
@@
 		(pts
 			(xy 72.39 88.9) (xy 72.39 83.82)
+		)
+		(stroke
+			(width 0)
+			(type default)
+		)
+	)
+	(wire
+		(pts
+			(xy 96.52 82.55) (xy 96.52 83.82)
 		)
 		(stroke
@@
 		(dnp no)
 		(fields_autoplaced yes)
-		(property "Reference" "D1"
+		(property "Reference" "D3"
 			(at 129.54 66.0399 90)
 			(effects
@@
 		(dnp no)
 		(fields_autoplaced yes)
-		(property "Reference" "C1"
+		(property "Reference" "C7"
 			(at 67.31 77.4699 0)
 			(effects
@@
 				(path "/acabfe98-929d-44a8-a67c-4204ca98f09f/ebcb53f7-58fd-409c-8719-320b24457066"
 					(reference "C4")
+					(unit 1)
+				)
+			)
+		)
+	)
+	(symbol
+		(lib_id "power:PWR_FLAG")
+		(at 189.23 74.93 0)
+		(unit 1)
+		(exclude_from_sim no)
+		(in_bom yes)
+		(on_board yes)
+		(dnp no)
+		(fields_autoplaced yes)
+		(property "Reference" "#FLG04"
+			(at 189.23 73.025 0)
+			(effects
+				(font
+					(size 1.27 1.27)
+				)
+				(hide yes)
+			)
+		)
+		(property "Value" "PWR_FLAG"
+			(at 189.23 69.85 0)
+			(effects
+				(font
+					(size 1.27 1.27)
+				)
+			)
+		)
+		(property "Footprint" ""
+			(at 189.23 74.93 0)
+			(effects
+				(font
+					(size 1.27 1.27)
+				)
+				(hide yes)
+			)
+		)
+		(property "Datasheet" "~"
+			(at 189.23 74.93 0)
+			(effects
+				(font
+					(size 1.27 1.27)
+				)
+				(hide yes)
+			)
+		)
+		(property "Description" "Special symbol for telling ERC where power comes from"
+			(at 189.23 74.93 0)
+			(effects
+				(font
+					(size 1.27 1.27)
+				)
+				(hide yes)
+			)
+		)
+		(pin "1"
+		)
+		(instances
+			(project "chessboard2"
+				(path "/acabfe98-929d-44a8-a67c-4204ca98f09f/baa1ed7e-b023-44da-b1f7-17a389052799"
+					(reference "#FLG04")
+					(unit 1)
+				)
+				(path "/acabfe98-929d-44a8-a67c-4204ca98f09f/ebcb53f7-58fd-409c-8719-320b24457066"
+					(reference "#FLG05")
+					(unit 1)
+				)
+				(path "/acabfe98-929d-44a8-a67c-4204ca98f09f/23ed26b1-8d60-43ca-b6a7-5586453700e2"
+					(reference "#FLG06")
+					(unit 1)
+				)
+				(path "/acabfe98-929d-44a8-a67c-4204ca98f09f/ea4f5474-c124-483a-b05c-97db30728daf"
+					(reference "#FLG07")
+					(unit 1)
+				)
+				(path "/acabfe98-929d-44a8-a67c-4204ca98f09f/8dc5d56a-bfdc-4a40-b66e-dfea5278dc65"
+					(reference "#FLG08")
+					(unit 1)
+				)
+				(path "/acabfe98-929d-44a8-a67c-4204ca98f09f/730ed345-c18d-4f02-adc8-c8506f5407de"
+					(reference "#FLG09")
+					(unit 1)
+				)
+				(path "/acabfe98-929d-44a8-a67c-4204ca98f09f/5a95ed4a-0e33-40ab-8120-c7c932b67184"
+					(reference "#FLG010")
+					(unit 1)
+				)
+				(path "/acabfe98-929d-44a8-a67c-4204ca98f09f/72d5fca6-10ec-41c2-be98-438aeffd8b3b"
+					(reference "#FLG011")
 					(unit 1)
 				)
@@
 		(dnp no)
 		(fields_autoplaced yes)
-		(property "Reference" "#PWR02"
+		(property "Reference" "#PWR010"
 			(at 135.89 109.22 0)
 			(effects
@@
 				(path "/acabfe98-929d-44a8-a67c-4204ca98f09f/ebcb53f7-58fd-409c-8719-320b24457066"
 					(reference "#PWR07")
+					(unit 1)
+				)
+			)
+		)
+	)
+	(symbol
+		(lib_id "power:PWR_FLAG")
+		(at 96.52 82.55 90)
+		(unit 1)
+		(exclude_from_sim no)
+		(in_bom yes)
+		(on_board yes)
+		(dnp no)
+		(fields_autoplaced yes)
+		(property "Reference" "#FLG012"
+			(at 94.615 82.55 0)
+			(effects
+				(font
+					(size 1.27 1.27)
+				)
+				(hide yes)
+			)
+		)
+		(property "Value" "PWR_FLAG"
+			(at 92.71 82.5499 90)
+			(effects
+				(font
+					(size 1.27 1.27)
+				)
+				(justify left)
+			)
+		)
+		(property "Footprint" ""
+			(at 96.52 82.55 0)
+			(effects
+				(font
+					(size 1.27 1.27)
+				)
+				(hide yes)
+			)
+		)
+		(property "Datasheet" "~"
+			(at 96.52 82.55 0)
+			(effects
+				(font
+					(size 1.27 1.27)
+				)
+				(hide yes)
+			)
+		)
+		(property "Description" "Special symbol for telling ERC where power comes from"
+			(at 96.52 82.55 0)
+			(effects
+				(font
+					(size 1.27 1.27)
+				)
+				(hide yes)
+			)
+		)
+		(pin "1"
+		)
+		(instances
+			(project "chessboard2"
+				(path "/acabfe98-929d-44a8-a67c-4204ca98f09f/baa1ed7e-b023-44da-b1f7-17a389052799"
+					(reference "#FLG012")
+					(unit 1)
+				)
+				(path "/acabfe98-929d-44a8-a67c-4204ca98f09f/ebcb53f7-58fd-409c-8719-320b24457066"
+					(reference "#FLG013")
+					(unit 1)
+				)
+				(path "/acabfe98-929d-44a8-a67c-4204ca98f09f/23ed26b1-8d60-43ca-b6a7-5586453700e2"
+					(reference "#FLG014")
+					(unit 1)
+				)
+				(path "/acabfe98-929d-44a8-a67c-4204ca98f09f/ea4f5474-c124-483a-b05c-97db30728daf"
+					(reference "#FLG015")
+					(unit 1)
+				)
+				(path "/acabfe98-929d-44a8-a67c-4204ca98f09f/8dc5d56a-bfdc-4a40-b66e-dfea5278dc65"
+					(reference "#FLG016")
+					(unit 1)
+				)
+				(path "/acabfe98-929d-44a8-a67c-4204ca98f09f/730ed345-c18d-4f02-adc8-c8506f5407de"
+					(reference "#FLG017")
+					(unit 1)
+				)
+				(path "/acabfe98-929d-44a8-a67c-4204ca98f09f/5a95ed4a-0e33-40ab-8120-c7c932b67184"
+					(reference "#FLG018")
+					(unit 1)
+				)
+				(path "/acabfe98-929d-44a8-a67c-4204ca98f09f/72d5fca6-10ec-41c2-be98-438aeffd8b3b"
+					(reference "#FLG019")
 					(unit 1)
 				)
@@
 		(dnp no)
 		(fields_autoplaced yes)
-		(property "Reference" "R1"
+		(property "Reference" "R5"
 			(at 99.06 76.1999 0)
 			(effects
@@
 		(dnp no)
 		(fields_autoplaced yes)
-		(property "Reference" "U1"
+		(property "Reference" "U5"
 			(at 98.7141 85.09 0)
 			(effects
@@
 			)
 		)
-		(property "Footprint" "Package_TO_SOT_SMD:SOT-23-8_Handsoldering"
+		(property "Footprint" "0chessbot:FSOP-8"
 			(at 88.9 91.44 0)
 			(effects
@@
 		(on_board yes)
 		(dnp no)
-		(property "Reference" "#PWR01"
+		(property "Reference" "#PWR09"
 			(at 120.65 59.69 0)
 			(effects
@@
 		(on_board yes)
 		(dnp no)
-		(property "Reference" "Q1"
+		(property "Reference" "Q3"
 			(at 168.91 71.1201 0)
 			(effects
@@
 		(dnp no)
 		(fields_autoplaced yes)
-		(property "Reference" "#PWR03"
+		(property "Reference" "#PWR011"
 			(at 165.1 60.96 0)
 			(effects
@@
 		(dnp no)
 		(fields_autoplaced yes)
-		(property "Reference" "C2"
+		(property "Reference" "C8"
 			(at 76.2 91.4399 0)
 			(effects
@@
 		(dnp no)
 		(fields_autoplaced yes)
-		(property "Reference" "C3"
+		(property "Reference" "C9"
 			(at 193.04 85.0899 0)
 			(effects
@@
 		(on_board yes)
 		(dnp no)
-		(property "Reference" "R2"
+		(property "Reference" "R6"
 			(at 142.24 62.2299 0)
 			(effects
@@
 		(dnp no)
 		(fields_autoplaced yes)
-		(property "Reference" "U2"
+		(property "Reference" "U6"
 			(at 172.72 85.0899 0)
 			(effects

Commit message: fix chessboard5 for ordering;
Parts:
- removed D3: LED_ARGB, LED_SMD:LED_Inolux_IN-PI554FCH_PLCC4_5.0x5.0mm_P3.2mm, symbol Device:LED_ARGB
- added D11: LED_RGAB, LED_SMD:LED_RGB_Wuerth-PLCC4_3.2x2.8mm_150141M173100, symbol Device:LED_GBRA
- C7, C8, C9: got (none) -> CL10A105KB8NNNC; gotnum (none) -> 600
- Q3: got (none) -> AO3401A; gotnum (none) -> 100
- R5: got (none) -> RC0603FR-07100RL; gotnum (none) -> 1000
- R6: got (none) -> RC0603FR-0710KL; gotnum (none) -> 1000
- U5: got (none) -> WS2814F; gotnum (none) -> 100
- U6: got (none) -> TMAG5273A2QDBVR; gotnum (none) -> 100
Connections:
- net +5V: now also D11.4 (A)
- net at U5.1 (OUTR): now also D11.3 (RK)
- net at U5.2 (OUTG): now also D11.2 (BK)
- net at U5.3 (OUTB): now also D11.1 (GK)
Changed lines of the file:
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@@
-	(wire
-		(pts
-			(xy 125.73 72.39) (xy 125.73 96.52)
-		)
-		(stroke
-			(width 0)
-			(type default)
-		)
-	)
 	(wire
 		(pts
@@
 	(wire
 		(pts
-			(xy 106.68 93.98) (xy 120.65 93.98)
-		)
-		(stroke
-			(width 0)
-			(type default)
-		)
-	)
-	(wire
-		(pts
 			(xy 135.89 102.87) (xy 165.1 102.87)
 		)
@@
 	(wire
 		(pts
-			(xy 106.68 91.44) (xy 115.57 91.44)
-		)
-		(stroke
-			(width 0)
-			(type default)
-		)
-	)
-	(wire
-		(pts
 			(xy 165.1 97.79) (xy 167.64 97.79)
 		)
@@
 	(wire
 		(pts
+			(xy 106.68 96.52) (xy 120.65 96.52)
+		)
+		(stroke
+			(width 0)
+			(type default)
+		)
+	)
+	(wire
+		(pts
 			(xy 120.65 57.15) (xy 120.65 62.23)
 		)
@@
 	(wire
 		(pts
-			(xy 106.68 96.52) (xy 125.73 96.52)
-		)
-		(stroke
-			(width 0)
-			(type default)
-		)
-	)
-	(wire
-		(pts
 			(xy 96.52 57.15) (xy 120.65 57.15)
 		)
@@
 	(wire
 		(pts
+			(xy 115.57 91.44) (xy 106.68 91.44)
+		)
+		(stroke
+			(width 0)
+			(type default)
+		)
+	)
+	(wire
+		(pts
+			(xy 115.57 72.39) (xy 115.57 91.44)
+		)
+		(stroke
+			(width 0)
+			(type default)
+		)
+	)
+	(wire
+		(pts
 			(xy 96.52 102.87) (xy 135.89 102.87)
 		)
@@
 	(wire
 		(pts
-			(xy 120.65 72.39) (xy 120.65 93.98)
+			(xy 120.65 72.39) (xy 120.65 96.52)
+		)
+		(stroke
+			(width 0)
+			(type default)
+		)
+	)
+	(wire
+		(pts
+			(xy 125.73 72.39) (xy 125.73 93.98)
 		)
 		(stroke
@@
 	(wire
 		(pts
+			(xy 125.73 93.98) (xy 106.68 93.98)
+		)
+		(stroke
+			(width 0)
+			(type default)
+		)
+	)
+	(wire
+		(pts
 			(xy 139.7 59.69) (xy 165.1 59.69)
 		)
@@
 		(pts
 			(xy 96.52 57.15) (xy 96.52 73.66)
-		)
-		(stroke
-			(width 0)
-			(type default)
-		)
-	)
-	(wire
-		(pts
-			(xy 115.57 72.39) (xy 115.57 91.44)
 		)
 		(stroke
@@
 	)
 	(symbol
-		(lib_id "Device:LED_ARGB")
+		(lib_id "Device:LED_GBRA")
 		(at 120.65 67.31 90)
 		(unit 1)
@@
 		(dnp no)
 		(fields_autoplaced yes)
-		(property "Reference" "D3"
+		(property "Reference" "D11"
 			(at 129.54 66.0399 90)
 			(effects
@@
 			)
 		)
-		(property "Value" "LED_ARGB"
+		(property "Value" "LED_RGAB"
 			(at 129.54 68.5799 90)
 			(effects
@@
 			)
 		)
-		(property "Footprint" "LED_SMD:LED_Inolux_IN-PI554FCH_PLCC4_5.0x5.0mm_P3.2mm"
+		(property "Footprint" "LED_SMD:LED_RGB_Wuerth-PLCC4_3.2x2.8mm_150141M173100"
 			(at 121.92 67.31 0)
 			(effects
@@
 			)
 		)
-		(property "Description" "RGB LED, anode/red/green/blue"
+		(property "Description" "RGB LED, green/blue/red/anode"
 			(at 120.65 67.31 0)
 			(effects
@@
 			)
 		)
+		(property "got" "XINGLIGHT XL-3227RGB-RF"
+			(at 120.65 67.31 0)
+			(effects
+				(font
+					(size 1.27 1.27)
+				)
+				(hide yes)
+			)
+		)
+		(property "gotnum" "100"
+			(at 120.65 67.31 0)
+			(effects
+				(font
+					(size 1.27 1.27)
+				)
+				(hide yes)
+			)
+		)
+		(pin "3"
+		)
+		(pin "2"
+		)
+		(pin "4"
+		)
 		(pin "1"
-		)
-		(pin "2"
-		)
-		(pin "3"
-		)
-		(pin "4"
 		)
 		(instances
 			(project "chessboard2"
 				(path "/acabfe98-929d-44a8-a67c-4204ca98f09f/23ed26b1-8d60-43ca-b6a7-5586453700e2"
-					(reference "D3")
+					(reference "D11")
+					(unit 1)
+				)
+				(path "/acabfe98-929d-44a8-a67c-4204ca98f09f/baa1ed7e-b023-44da-b1f7-17a389052799"
+					(reference "D9")
+					(unit 1)
+				)
+				(path "/acabfe98-929d-44a8-a67c-4204ca98f09f/ebcb53f7-58fd-409c-8719-320b24457066"
+					(reference "D10")
+					(unit 1)
+				)
+				(path "/acabfe98-929d-44a8-a67c-4204ca98f09f/ea4f5474-c124-483a-b05c-97db30728daf"
+					(reference "D12")
+					(unit 1)
+				)
+				(path "/acabfe98-929d-44a8-a67c-4204ca98f09f/8dc5d56a-bfdc-4a40-b66e-dfea5278dc65"
+					(reference "D13")
+					(unit 1)
+				)
+				(path "/acabfe98-929d-44a8-a67c-4204ca98f09f/730ed345-c18d-4f02-adc8-c8506f5407de"
+					(reference "D14")
 					(unit 1)
 				)
 				(path "/acabfe98-929d-44a8-a67c-4204ca98f09f/5a95ed4a-0e33-40ab-8120-c7c932b67184"
-					(reference "D7")
+					(reference "D15")
 					(unit 1)
 				)
 				(path "/acabfe98-929d-44a8-a67c-4204ca98f09f/72d5fca6-10ec-41c2-be98-438aeffd8b3b"
-					(reference "D8")
-					(unit 1)
-				)
-				(path "/acabfe98-929d-44a8-a67c-4204ca98f09f/730ed345-c18d-4f02-adc8-c8506f5407de"
-					(reference "D6")
-					(unit 1)
-				)
-				(path "/acabfe98-929d-44a8-a67c-4204ca98f09f/8dc5d56a-bfdc-4a40-b66e-dfea5278dc65"
-					(reference "D5")
-					(unit 1)
-				)
-				(path "/acabfe98-929d-44a8-a67c-4204ca98f09f/baa1ed7e-b023-44da-b1f7-17a389052799"
-					(reference "D1")
-					(unit 1)
-				)
-				(path "/acabfe98-929d-44a8-a67c-4204ca98f09f/ea4f5474-c124-483a-b05c-97db30728daf"
-					(reference "D4")
-					(unit 1)
-				)
-				(path "/acabfe98-929d-44a8-a67c-4204ca98f09f/ebcb53f7-58fd-409c-8719-320b24457066"
-					(reference "D2")
+					(reference "D16")
 					(unit 1)
 				)
@@
 			)
 		)
+		(property "got" "CL10A105KB8NNNC"
+			(at 63.5 78.74 0)
+			(effects
+				(font
+					(size 1.27 1.27)
+				)
+				(hide yes)
+			)
+		)
+		(property "gotnum" "600"
+			(at 63.5 78.74 0)
+			(effects
+				(font
+					(size 1.27 1.27)
+				)
+				(hide yes)
+			)
+		)
 		(pin "1"
 		)
@@
 			)
 		)
+		(property "got" " RC0603FR-07100RL"
+			(at 96.52 77.47 0)
+			(effects
+				(font
+					(size 1.27 1.27)
+				)
+				(hide yes)
+			)
+		)
+		(property "gotnum" "1000"
+			(at 96.52 77.47 0)
+			(effects
+				(font
+					(size 1.27 1.27)
+				)
+				(hide yes)
+			)
+		)
 		(pin "1"
 		)
@@
 			)
 		)
+		(property "got" "WS2814F"
+			(at 96.52 95.25 0)
+			(effects
+				(font
+					(size 1.27 1.27)
+				)
+				(hide yes)
+			)
+		)
+		(property "gotnum" "100"
+			(at 96.52 95.25 0)
+			(effects
+				(font
+					(size 1.27 1.27)
+				)
+				(hide yes)
+			)
+		)
 		(pin "8"
 		)
@@
 			)
 		)
+		(property "got" "AO3401A"
+			(at 162.56 69.85 0)
+			(effects
+				(font
+					(size 1.27 1.27)
+				)
+				(hide yes)
+			)
+		)
+		(property "gotnum" "100"
+			(at 162.56 69.85 0)
+			(effects
+				(font
+					(size 1.27 1.27)
+				)
+				(hide yes)
+			)
+		)
 		(pin "2"
 		)
@@
 			)
 		)
+		(property "got" "CL10A105KB8NNNC"
+			(at 72.39 92.71 0)
+			(effects
+				(font
+					(size 1.27 1.27)
+				)
+				(hide yes)
+			)
+		)
+		(property "gotnum" "600"
+			(at 72.39 92.71 0)
+			(effects
+				(font
+					(size 1.27 1.27)
+				)
+				(hide yes)
+			)
+		)
 		(pin "1"
 		)
@@
 			)
 		)
+		(property "got" "CL10A105KB8NNNC"
+			(at 189.23 86.36 0)
+			(effects
+				(font
+					(size 1.27 1.27)
+				)
+				(hide yes)
+			)
+		)
+		(property "gotnum" "600"
+			(at 189.23 86.36 0)
+			(effects
+				(font
+					(size 1.27 1.27)
+				)
+				(hide yes)
+			)
+		)
 		(pin "1"
 		)
@@
 		)
 		(property "Description" "Resistor"
+			(at 139.7 63.5 0)
+			(effects
+				(font
+					(size 1.27 1.27)
+				)
+				(hide yes)
+			)
+		)
+		(property "got" " RC0603FR-0710KL"
+			(at 139.7 63.5 0)
+			(effects
+				(font
+					(size 1.27 1.27)
+				)
+				(hide yes)
+			)
+		)
+		(property "gotnum" "1000"
 			(at 139.7 63.5 0)
 			(effects
@@
 			(at 165.1 87.63 0)
 			(effects
+				(font
+					(size 1.27 1.27)
+				)
+				(hide yes)
+			)
+		)
+		(property "got" "TMAG5273A2QDBVR"
+			(at 165.1 87.63 0)
+			(effects
+				(font
+					(size 1.27 1.27)
+				)
+				(hide yes)
+			)
+		)
+		(property "gotnum" "100"
+			(at 165.1 87.63 0)
+			(effects
