File: chessboard5/chessboard2.kicad_pcb (KiCad board)
At the start: 2 copper layers, 54.4 x 12.5 mm, 13 parts, among them J1 IN, J2 OUT, J3 IN, J4 OUT, Q1 AP2003 P/NMOS Pair, U1 TMAG5273, U2 WS2814F

Commit message: fix up schematic for chessboard5
Parts:
- removed J1, J3: IN, Connector_PinSocket_2.54mm:PinSocket_1x05_P2.54mm_Vertical
- removed J2, J4: OUT, Connector_PinHeader_2.54mm:PinHeader_1x05_P2.54mm_Vertical
- removed REF**: LED_Avago_PLCC4_3.2x2.8mm_CW, LED_SMD:LED_Avago_PLCC4_3.2x2.8mm_CW
- added C10: 1u, Capacitor_SMD:C_0603_1608Metric_Pad1.08x0.95mm_HandSolder, F.Cu at (104.0, 71.2)
- added C11: 1u, Capacitor_SMD:C_0603_1608Metric_Pad1.08x0.95mm_HandSolder, F.Cu at (104.0, 73.7)
- added C12: 1u, Capacitor_SMD:C_0603_1608Metric_Pad1.08x0.95mm_HandSolder, F.Cu at (104.0, 76.2)
- added C13: 1u, Capacitor_SMD:C_0603_1608Metric_Pad1.08x0.95mm_HandSolder, F.Cu at (67.9, 89.3)
- added C14: 1u, Capacitor_SMD:C_0603_1608Metric_Pad1.08x0.95mm_HandSolder, F.Cu at (67.9, 91.8)
- added C15: 1u, Capacitor_SMD:C_0603_1608Metric_Pad1.08x0.95mm_HandSolder, F.Cu at (67.9, 94.3)
- added C16: 1u, Capacitor_SMD:C_0603_1608Metric_Pad1.08x0.95mm_HandSolder, F.Cu at (67.9, 71.2)
- added C17: 1u, Capacitor_SMD:C_0603_1608Metric_Pad1.08x0.95mm_HandSolder, F.Cu at (67.9, 73.7)
- added C18: 1u, Capacitor_SMD:C_0603_1608Metric_Pad1.08x0.95mm_HandSolder, F.Cu at (67.9, 76.2)
- added C19: 1u, Capacitor_SMD:C_0603_1608Metric_Pad1.08x0.95mm_HandSolder, F.Cu at (86.0, 53.1)
- added C2: 1u, Capacitor_SMD:C_0603_1608Metric_Pad1.08x0.95mm_HandSolder, F.Cu at (86.0, 73.7)
- added C20: 1u, Capacitor_SMD:C_0603_1608Metric_Pad1.08x0.95mm_HandSolder, F.Cu at (86.0, 55.6)
- added C21: 1u, Capacitor_SMD:C_0603_1608Metric_Pad1.08x0.95mm_HandSolder, F.Cu at (86.0, 58.1)
- added C22: 1u, Capacitor_SMD:C_0603_1608Metric_Pad1.08x0.95mm_HandSolder, F.Cu at (104.0, 53.1)
- added C23: 1u, Capacitor_SMD:C_0603_1608Metric_Pad1.08x0.95mm_HandSolder, F.Cu at (104.0, 55.6)
- added C24: 1u, Capacitor_SMD:C_0603_1608Metric_Pad1.08x0.95mm_HandSolder, F.Cu at (104.0, 58.1)
- added C3: 1u, Capacitor_SMD:C_0603_1608Metric_Pad1.08x0.95mm_HandSolder, F.Cu at (86.0, 76.2)
- added C4: 1u, Capacitor_SMD:C_0603_1608Metric_Pad1.08x0.95mm_HandSolder, F.Cu at (86.0, 89.3)
- added C5: 1u, Capacitor_SMD:C_0603_1608Metric_Pad1.08x0.95mm_HandSolder, F.Cu at (86.0, 91.8)
- added C6: 1u, Capacitor_SMD:C_0603_1608Metric_Pad1.08x0.95mm_HandSolder, F.Cu at (86.0, 94.3)
- added C7: 1u, Capacitor_SMD:C_0603_1608Metric_Pad1.08x0.95mm_HandSolder, F.Cu at (67.9, 53.1)
- added C8: 1u, Capacitor_SMD:C_0603_1608Metric_Pad1.08x0.95mm_HandSolder, F.Cu at (67.9, 55.6)
- added C9: 1u, Capacitor_SMD:C_0603_1608Metric_Pad1.08x0.95mm_HandSolder, F.Cu at (67.9, 58.1)
- added D2: LED_ARGB, LED_SMD:LED_Inolux_IN-PI554FCH_PLCC4_5.0x5.0mm_P3.2mm, F.Cu at (92.1, 91.3)
- added D3: LED_ARGB, LED_SMD:LED_Inolux_IN-PI554FCH_PLCC4_5.0x5.0mm_P3.2mm, F.Cu at (74.1, 55.1)
- added D4: LED_ARGB, LED_SMD:LED_Inolux_IN-PI554FCH_PLCC4_5.0x5.0mm_P3.2mm, F.Cu at (110.2, 73.2)
- added D5: LED_ARGB, LED_SMD:LED_Inolux_IN-PI554FCH_PLCC4_5.0x5.0mm_P3.2mm, F.Cu at (74.1, 91.3)
- added D6: LED_ARGB, LED_SMD:LED_Inolux_IN-PI554FCH_PLCC4_5.0x5.0mm_P3.2mm, F.Cu at (74.1, 73.2)
- added D7: LED_ARGB, LED_SMD:LED_Inolux_IN-PI554FCH_PLCC4_5.0x5.0mm_P3.2mm, F.Cu at (92.1, 55.1)
- added D8: LED_ARGB, LED_SMD:LED_Inolux_IN-PI554FCH_PLCC4_5.0x5.0mm_P3.2mm, F.Cu at (110.2, 55.1)
- added Q2: AO3401A, Package_TO_SOT_SMD:SOT-23_Handsoldering, F.Cu at (91.4, 97.1)
- added Q3: AO3401A, Package_TO_SOT_SMD:SOT-23_Handsoldering, F.Cu at (73.3, 60.9)
- added Q4: AO3401A, Package_TO_SOT_SMD:SOT-23_Handsoldering, F.Cu at (109.4, 79.0)
- added Q5: AO3401A, Package_TO_SOT_SMD:SOT-23_Handsoldering, F.Cu at (73.3, 97.1)
- added Q6: AO3401A, Package_TO_SOT_SMD:SOT-23_Handsoldering, F.Cu at (73.3, 79.0)
- added Q7: AO3401A, Package_TO_SOT_SMD:SOT-23_Handsoldering, F.Cu at (91.4, 60.9)
- added Q8: AO3401A, Package_TO_SOT_SMD:SOT-23_Handsoldering, F.Cu at (109.4, 60.9)
- added R10: 10k, Resistor_SMD:R_0603_1608Metric_Pad0.98x0.95mm_HandSolder, F.Cu at (67.9, 99.3)
- added R11: 100R, Resistor_SMD:R_0603_1608Metric_Pad0.98x0.95mm_HandSolder, F.Cu at (67.9, 78.7)
- added R12: 10k, Resistor_SMD:R_0603_1608Metric_Pad0.98x0.95mm_HandSolder, F.Cu at (67.9, 81.3)
- added R13: 100R, Resistor_SMD:R_0603_1608Metric_Pad0.98x0.95mm_HandSolder, F.Cu at (86.0, 60.7)
- added R14: 10k, Resistor_SMD:R_0603_1608Metric_Pad0.98x0.95mm_HandSolder, F.Cu at (86.0, 63.2)
- added R15: 100R, Resistor_SMD:R_0603_1608Metric_Pad0.98x0.95mm_HandSolder, F.Cu at (104.0, 60.7)
- added R16: 10k, Resistor_SMD:R_0603_1608Metric_Pad0.98x0.95mm_HandSolder, F.Cu at (104.0, 63.2)
- added R17: 100R, Resistor_SMD:R_0603_1608Metric_Pad0.98x0.95mm_HandSolder, F.Cu at (104.0, 89.3)
- added R4: 10k, Resistor_SMD:R_0603_1608Metric_Pad0.98x0.95mm_HandSolder, F.Cu at (86.0, 99.3)
- added R5: 100R, Resistor_SMD:R_0603_1608Metric_Pad0.98x0.95mm_HandSolder, F.Cu at (67.9, 60.7)
- added R6: 10k, Resistor_SMD:R_0603_1608Metric_Pad0.98x0.95mm_HandSolder, F.Cu at (67.9, 63.2)
- added R7: 100R, Resistor_SMD:R_0603_1608Metric_Pad0.98x0.95mm_HandSolder, F.Cu at (104.0, 78.7)
- added R8: 10k, Resistor_SMD:R_0603_1608Metric_Pad0.98x0.95mm_HandSolder, F.Cu at (104.0, 81.3)
- added R9: 100R, Resistor_SMD:R_0603_1608Metric_Pad0.98x0.95mm_HandSolder, F.Cu at (67.9, 96.8)
- added U10: TMAG5273, Package_TO_SOT_SMD:SOT-23-6_Handsoldering, F.Cu at (78.9, 101.8)
- added U11: WS2814F, Package_TO_SOT_SMD:SOT-23-8_Handsoldering, F.Cu at (73.0, 83.7)
- added U12: TMAG5273, Package_TO_SOT_SMD:SOT-23-6_Handsoldering, F.Cu at (78.9, 83.7)
- added U13: WS2814F, Package_TO_SOT_SMD:SOT-23-8_Handsoldering, F.Cu at (91.1, 65.6)
- added U14: TMAG5273, Package_TO_SOT_SMD:SOT-23-6_Handsoldering, F.Cu at (96.9, 65.6)
- added U15: WS2814F, Package_TO_SOT_SMD:SOT-23-8_Handsoldering, F.Cu at (109.1, 65.6)
- added U16: TMAG5273, Package_TO_SOT_SMD:SOT-23-6_Handsoldering, F.Cu at (115.0, 65.6)
- added U3: WS2814F, Package_TO_SOT_SMD:SOT-23-8_Handsoldering, F.Cu at (91.1, 101.8)
- added U4: TMAG5273, Package_TO_SOT_SMD:SOT-23-6_Handsoldering, F.Cu at (96.9, 101.8)
- added U5: WS2814F, Package_TO_SOT_SMD:SOT-23-8_Handsoldering, F.Cu at (73.0, 65.6)
- added U6: TMAG5273, Package_TO_SOT_SMD:SOT-23-6_Handsoldering, F.Cu at (78.9, 65.6)
- added U7: WS2814F, Package_TO_SOT_SMD:SOT-23-8_Handsoldering, F.Cu at (109.1, 83.7)
- added U8: TMAG5273, Package_TO_SOT_SMD:SOT-23-6_Handsoldering, F.Cu at (115.0, 83.7)
- added U9: WS2814F, Package_TO_SOT_SMD:SOT-23-8_Handsoldering, F.Cu at (73.0, 101.8)
- C1: value 100n -> 1u
- D1: value LED_RGB -> LED_ARGB; footprint LED_SMD:LED_RGB_5050-6 -> LED_SMD:LED_Inolux_IN-PI554FCH_PLCC4_5.0x5.0mm_P3.2mm
- Q1: value AP2003 P/NMOS Pair -> AO3401A; footprint Package_TO_SOT_SMD:SOT-23-6_Handsoldering -> Package_TO_SOT_SMD:SOT-23_Handsoldering
- R1, R3: value 200 -> 100R
- U1: value TMAG5273 -> WS2814F; footprint Package_TO_SOT_SMD:SOT-23-6 -> Package_TO_SOT_SMD:SOT-23-8_Handsoldering
- U2: value WS2814F -> TMAG5273; footprint Package_TO_SOT_SMD:SOT-23-8_Handsoldering -> Package_TO_SOT_SMD:SOT-23-6_Handsoldering
- moved R1 46.5 mm to (86.0, 78.7), turned to 0 degrees
- moved D1 45.9 mm to (92.1, 73.2)
- moved C1 43.5 mm to (86.0, 71.2)
- moved R2 36.6 mm to (86.0, 81.3)
- moved Q1 34.1 mm to (91.4, 79.0), turned to 0 degrees
- moved U1 32.4 mm to (91.1, 83.7), turned to 0 degrees
- moved U2 31.7 mm to (96.9, 83.7), turned to 0 degrees
- moved R3 22.2 mm to (86.0, 96.8), turned to 0 degrees
Connections:
- C1 pad 1: Net-(Q1B-DP) -> 5V
- D1 pad 1: Net-(D1-RK) -> 5V
- D1 pad 2: Net-(D1-GK) -> Net-(D1-RK)
- D1 pad 3: Net-(D1-BK) -> Net-(D1-GK)
- D1 pad 4: VCC -> Net-(D1-BK)
- Q1 pad 1: GND -> Net-(Q1-G)
- Q1 pad 2: Net-(Q1A-GN) -> +3V3
- Q1 pad 3: Net-(Q1B-DP) -> Net-(Q1-D)
- R1 pad 1: DIN -> 5V
- R1 pad 2: Net-(U2-DIN) -> Net-(U1-VDD)
- R2 pad 1: Net-(Q1A-DN) -> Net-(Q1-G)
- R2 pad 2: VCC -> +3V3
- R3 pad 1: Net-(Q1A-GN) -> 5V
- R3 pad 2: VCC -> Net-(U3-VDD)
- U1 pad 1: SDA -> Net-(D1-RK)
- U1 pad 2: GND -> Net-(D1-GK)
- U1 pad 3: GND -> Net-(D1-BK)
- U1 pad 4: Net-(Q1B-DP) -> GND
- U1 pad 5: GND -> /Cell/DOUT
- U1 pad 6: SCL -> /Cell/DIN
- U2 pad 1: Net-(D1-GK) -> SDA
- U2 pad 2: Net-(D1-RK) -> GND
- U2 pad 3: Net-(D1-BK) -> GND
- U2 pad 4: GND -> Net-(Q1-D)
- U2 pad 5: DOUT -> GND
- U2 pad 6: Net-(U2-DIN) -> SCL
Routing:
- net VCC: track 71.8 -> 0.00 mm, vias 1 -> 0
- net GND: track 51.4 -> 0.00 mm
- net SCL: track 47.4 -> 0.00 mm, vias 1 -> 0
- net SDA: track 41.5 -> 0.00 mm, vias 1 -> 0
- net DOUT: track 18.4 -> 0.00 mm, vias 1 -> 0
- net DIN: track 16.9 -> 0.00 mm
- net Net-(D1-BK): track 10.3 -> 0.00 mm
- net Net-(D1-RK): track 10.2 -> 0.00 mm
- net Net-(D1-GK): track 7.99 -> 0.00 mm
- net Net-(U2-DIN): track 6.57 -> 0.00 mm
- net Net-(Q1B-DP): track 3.76 -> 0.00 mm
- net Net-(Q1A-GN): track 3.71 -> 0.00 mm
- net Net-(Q1A-DN): track 2.68 -> 0.00 mm
Other:
- board size 54.4 x 12.5 mm -> 240 x 12 mm

Commit message: Progress!!!
Parts:
- added J1: Conn_01x06, Connector_IDC:IDC-Header_2x03_P2.54mm_Vertical, F.Cu at (287.5, 119.9)
- added J2: Conn_01x06, Connector_IDC:IDC-Header_2x03_P2.54mm_Vertical, F.Cu at (54.0, 120.0)
- moved C10 154.3 mm to (258.2, 65.2)
- moved C11 154.3 mm to (258.2, 67.8)
- moved C12 154.3 mm to (258.2, 70.3)
- moved C13 154.3 mm to (222.1, 83.3)
- moved C14 154.3 mm to (222.1, 85.8)
- moved C15 154.3 mm to (222.1, 88.4)
- moved C16 154.3 mm to (222.1, 65.2)
- moved C17 154.3 mm to (222.1, 67.8)
- moved C18 154.3 mm to (222.1, 70.3)
- moved C19 154.3 mm to (240.2, 47.2)
- moved C20 154.3 mm to (240.2, 49.7)
- moved C21 154.3 mm to (240.2, 52.2)
- moved C22 154.3 mm to (258.2, 47.2)
- moved C23 154.3 mm to (258.2, 49.7)
- moved C24 154.3 mm to (258.2, 52.2)
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Connections:
- net +3V3 renamed +3.3V
- net 5V renamed +5V
- C11 pad 2: unconnected-(C11-Pad2) -> GND
- C14 pad 2: unconnected-(C14-Pad2) -> GND
- C17 pad 2: unconnected-(C17-Pad2) -> GND
- C2 pad 2: unconnected-(C2-Pad2) -> GND
- C20 pad 2: unconnected-(C20-Pad2) -> GND
- C23 pad 2: unconnected-(C23-Pad2) -> GND
- C5 pad 2: unconnected-(C5-Pad2) -> GND
- C8 pad 2: unconnected-(C8-Pad2) -> GND
Routing:
- net GND: track 0.00 -> 292.7 mm, vias 0 -> 1
- net +5V: track 0.00 -> 242.1 mm, vias 0 -> 1
- net SCL: track 0.00 -> 241.8 mm, vias 0 -> 1
- net +3.3V: track 0.00 -> 238.7 mm
- net SDA: track 0.00 -> 237.1 mm, vias 0 -> 1
- net Net-(Q1-G): track 0.00 -> 22.4 mm
- net /Cell/DIN: track 0.00 -> 15.8 mm
- net Net-(D1-RK): track 0.00 -> 12.3 mm
- net Net-(D1-BK): track 0.00 -> 11.6 mm
- net Net-(J2-Pin_3): track 0.00 -> 7.85 mm
- net Net-(Q1-D): track 0.00 -> 7.71 mm
- net Net-(U1-VDD): track 0.00 -> 7.08 mm
- net Net-(D1-GK): track 0.00 -> 6.00 mm

Commit message: pcb progress 2
Parts:
- moved U4 156.9 mm to (97.0, 125.5)
- moved C6 144.2 mm to (101.0, 126.0), turned to 90 degrees
- moved Q2 143.7 mm to (106.0, 125.5), turned to 180 degrees
- moved U3 141.3 mm to (106.0, 120.0)
- moved R4 134.1 mm to (110.0, 125.5), turned to 90 degrees
- moved C5 131.4 mm to (113.0, 119.0)
- moved R3 130.6 mm to (113.1, 121.0), turned to 180 degrees
- moved C4 128.5 mm to (117.0, 120.0), turned to 90 degrees
- moved U6 124.8 mm to (127.0, 125.5)
- moved D3 123.6 mm to (127.0, 120.0)
- moved U8 121.9 mm to (157.0, 125.5)
- moved D4 119.6 mm to (157.0, 120.0)
- moved C9 117.3 mm to (131.0, 126.0), turned to 90 degrees
- moved Q3 115.5 mm to (136.0, 125.5), turned to 180 degrees
- moved C12 112.0 mm to (161.0, 126.0), turned to 90 degrees
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Routing:
- net GND: track 292.7 -> 562.6 mm, vias 1 -> 8
- net +5V: track 242.1 -> 366.8 mm, vias 1 -> 10
- net +3.3V: track 238.7 -> 351.9 mm, vias 0 -> 7
- net SCL: track 241.8 -> 283.0 mm, vias 1 -> 8
- net /Cell/DOUT: track 0.00 -> 36.3 mm, vias 0 -> 2
- net /Cell2/DOUT: track 0.00 -> 35.3 mm, vias 0 -> 2
- net /Cell5/DOUT: track 0.00 -> 31.7 mm, vias 0 -> 2
- net /Cell3/DOUT: track 0.00 -> 31.7 mm, vias 0 -> 2
- net /Cell4/DOUT: track 0.00 -> 31.6 mm, vias 0 -> 2
- net /Cell1/DOUT: track 0.00 -> 31.2 mm, vias 0 -> 2
- net Net-(U15-VDD): track 0.00 -> 28.2 mm, vias 0 -> 4
- net Net-(Q8-D): track 0.00 -> 25.3 mm, vias 0 -> 2
- net Net-(Q4-G): track 0.00 -> 22.4 mm
- net Net-(Q3-G): track 0.00 -> 22.4 mm
- net Net-(Q6-G): track 0.00 -> 22.4 mm
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
Commit message: finished chessboard v5!!!
Parts:
- added H1: MountingHole, MountingHole:MountingHole_3.2mm_M3, F.Cu at (149.0, 124.5)
- J1, J2: footprint Connector_IDC:IDC-Header_2x03_P2.54mm_Vertical -> Connector_PinHeader_2.54mm:PinHeader_2x03_P2.54mm_Vertical
- U1, U11, U13, U15, U3, U5, U7, U9: footprint Package_TO_SOT_SMD:SOT-23-8_Handsoldering -> 0chessbot:FSOP-8
- moved C7 1.00 mm to (146.0, 120.0)
- moved J1 0.09 mm to (287.5, 120.0)
Routing:
- net SDA: track 250.0 -> 256.3 mm
- net +5V: track 366.8 -> 368.4 mm
- net SCL: track 283.0 -> 284.4 mm
- net +3.3V: track 351.9 -> 352.7 mm
Other:
- board text added: "8x 0603 10kOhm Resistor (near mosfet) 9x 0603 100Ohm Resistor (everything else) 8x SOT-23-8 but .8mm WS2814F LED Driver 8x SOT-23-6 TMAG5273 Magnetometer"
- board text added: "By Barrett Lubianski"
- board text added: "By Karmanyaah Malhotra"
- board text added: "By Olyvia Witham"
- board text added: "Chessboard Row v5 UT Austin IEEE RAS Demobots - Chessbot https://github.com/ut-ras/chessbot Designed by Karmanyaah Malhotra, Olyvia Witham, Barrett Lubianski"
- board text added: "JLCJLCJLCJLC"
- board text added: "Parts: 24x 0603 1uF Capacitor 8x PLCC-4 5050 Com. Anode RGB LED 2x 2x03 2.54mm Connector"

Commit message: fix chessboard5 for ordering;
Parts:
- removed D1, D2, D3, D4, D5, D6, D7, D8: LED_ARGB, LED_SMD:LED_Inolux_IN-PI554FCH_PLCC4_5.0x5.0mm_P3.2mm
- added D10: LED_RGAB, LED_SMD:LED_RGB_Wuerth-PLCC4_3.2x2.8mm_150141M173100, F.Cu at (97.0, 119.8)
- added D11: LED_RGAB, LED_SMD:LED_RGB_Wuerth-PLCC4_3.2x2.8mm_150141M173100, F.Cu at (127.0, 119.8)
- added D12: LED_RGAB, LED_SMD:LED_RGB_Wuerth-PLCC4_3.2x2.8mm_150141M173100, F.Cu at (157.0, 119.8)
- added D13: LED_RGAB, LED_SMD:LED_RGB_Wuerth-PLCC4_3.2x2.8mm_150141M173100, F.Cu at (187.0, 119.8)
- added D14: LED_RGAB, LED_SMD:LED_RGB_Wuerth-PLCC4_3.2x2.8mm_150141M173100, F.Cu at (217.0, 119.8)
- added D15: LED_RGAB, LED_SMD:LED_RGB_Wuerth-PLCC4_3.2x2.8mm_150141M173100, F.Cu at (247.0, 119.8)
- added D16: LED_RGAB, LED_SMD:LED_RGB_Wuerth-PLCC4_3.2x2.8mm_150141M173100, F.Cu at (277.0, 119.8)
- added D9: LED_RGAB, LED_SMD:LED_RGB_Wuerth-PLCC4_3.2x2.8mm_150141M173100, F.Cu at (67.0, 119.8)
- added JP1: SolderJumper_3_Open, Jumper:SolderJumper-3_P1.3mm_Open_RoundedPad1.0x1.5mm, B.Cu at (61.4, 121.5)
- added JP2: SolderJumper_3_Open, Jumper:SolderJumper-3_P1.3mm_Open_RoundedPad1.0x1.5mm, B.Cu at (279.8, 121.5)
- moved H1 28.0 mm to (177.0, 125.0)
- moved C22 20.4 mm to (261.6, 126.2), turned to -90 degrees
- moved C23 18.8 mm to (265.3, 126.9), turned to 180 degrees
- moved C24 8.02 mm to (281.0, 126.1)
- moved Q8 3.27 mm to (271.7, 126.2), turned to 0 degrees
- moved R16 2.98 mm to (267.9, 126.2), turned to -90 degrees
- moved R15 2.51 mm to (265.2, 125.2), turned to 0 degrees
- moved U15 1.15 mm to (271.7, 121.0)
- moved R14 0.92 mm to (259.4, 126.2)
- moved R10 0.92 mm to (199.4, 126.2)
- moved R12 0.92 mm to (229.4, 126.2)
- moved R2 0.92 mm to (79.4, 126.2)
- moved R4 0.92 mm to (109.4, 126.2)
- moved R6 0.92 mm to (139.4, 126.2)
- moved R8 0.92 mm to (169.4, 126.2)
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Connections:
- J1 pad 3: /Cell7/DOUT -> Net-(J1-Pin_3)
- R17 pad 2: Net-(J2-Pin_3) -> /DIN_G
- U15 pad 5: /Cell7/DOUT -> /DOUT_G
Routing:
- net /DIN_G: track 0.00 -> 224.0 mm, vias 0 -> 2
- net /DOUT_G: track 0.00 -> 222.0 mm, vias 0 -> 1
- net +5V: track 368.4 -> 309.3 mm, vias 10 -> 16
- net GND: track 562.9 -> 513.3 mm, vias 8 -> 16
- net Net-(U15-VDD): track 28.4 -> 7.80 mm, vias 4 -> 0
- net /Cell7/DOUT: track 19.6 -> 0.00 mm, vias 2 -> 0
- net Net-(Q8-D): track 25.3 -> 9.24 mm, vias 2 -> 0
- net Net-(Q4-G): track 22.4 -> 13.3 mm
- net Net-(Q3-G): track 22.4 -> 13.3 mm
- net Net-(Q6-G): track 22.4 -> 13.3 mm
- net Net-(Q5-G): track 22.4 -> 13.3 mm
- net Net-(Q2-G): track 22.4 -> 13.3 mm
- net Net-(Q1-G): track 22.4 -> 13.3 mm
- net Net-(Q7-G): track 22.4 -> 13.3 mm
- net Net-(D16-GK): track 11.5 -> 2.46 mm
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