File: chessboard5-bus/chessboard5-bus.kicad_pcb (KiCad board)
At the start: 2 copper layers, 10 x 300 mm, 14 parts, among them J1 Conn_01x06, J10 Conn_01x06, J11 Conn_01x08, J2 Conn_01x06, J3 Conn_01x06, J4 Conn_01x06, J5 Conn_01x06, J6 Conn_01x06, J7 Conn_01x06, J8 Conn_01x06, J9 Conn_01x06

Commit message: fix chessboard5 for ordering;
Routing:
- net +3V3: vias 2 -> 5
- net GND: vias 5 -> 13
- net +5V: vias 4 -> 11
Changed lines of the file:
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@@
+	)
+	(via
+		(at 125.7 37)
+		(size 0.6)
+		(drill 0.3)
+		(layers "F.Cu" "B.Cu")
+		(free yes)
+		(net 1)
+	)
+	(via
+		(at 127.5 279)
+		(size 0.6)
+		(drill 0.3)
+		(layers "F.Cu" "B.Cu")
+		(free yes)
+		(net 1)
+	)
+	(via
+		(at 126.5 279)
+		(size 0.6)
+		(drill 0.3)
+		(layers "F.Cu" "B.Cu")
+		(free yes)
+		(net 1)
+	)
+	(via
+		(at 126.4 247)
+		(size 0.6)
+		(drill 0.3)
+		(layers "F.Cu" "B.Cu")
+		(free yes)
+		(net 1)
+	)
+	(via
+		(at 128.5 279)
+		(size 0.6)
+		(drill 0.3)
+		(layers "F.Cu" "B.Cu")
+		(free yes)
+		(net 1)
 	)
 	(via
@@
 	)
 	(via
+		(at 127.683977 247)
+		(size 0.6)
+		(drill 0.3)
+		(layers "F.Cu" "B.Cu")
+		(free yes)
+		(net 1)
+	)
+	(via
 		(at 129 15.5)
 		(size 0.6)
@@
 	(via
 		(at 129 17)
+		(size 0.6)
+		(drill 0.3)
+		(layers "F.Cu" "B.Cu")
+		(free yes)
+		(net 1)
+	)
+	(via
+		(at 127.5 37)
 		(size 0.6)
 		(drill 0.3)
@@
 	)
 	(via
+		(at 132.5 247)
+		(size 0.6)
+		(drill 0.3)
+		(layers "F.Cu" "B.Cu")
+		(free yes)
+		(net 4)
+	)
+	(via
+		(at 130 279)
+		(size 0.6)
+		(drill 0.3)
+		(layers "F.Cu" "B.Cu")
+		(free yes)
+		(net 4)
+	)
+	(via
 		(at 132.85 34)
 		(size 0.6)
@@
 		(drill 0.3)
 		(layers "F.Cu" "B.Cu")
+		(net 4)
+	)
+	(via
+		(at 128.5 37)
+		(size 0.6)
+		(drill 0.3)
+		(layers "F.Cu" "B.Cu")
+		(net 4)
+	)
+	(segment
+		(start 128.45 36.95)
+		(end 128.45 34.1)
+		(width 0.5)
+		(layer "B.Cu")
 		(net 4)
 	)
@@
 	)
 	(segment
+		(start 128.5 37)
+		(end 128.45 36.95)
+		(width 0.5)
+		(layer "B.Cu")
+		(net 4)
+	)
+	(segment
+		(start 128.45 37.05)
+		(end 128.5 37)
+		(width 0.5)
+		(layer "B.Cu")
+		(net 4)
+	)
+	(segment
 		(start 131.265 49.475)
 		(end 129.9 48.11)
@@
 	(segment
 		(start 128.45 41.95)
-		(end 128.45 34.1)
+		(end 128.45 37.05)
 		(width 0.5)
 		(layer "B.Cu")
@@
 	)
 	(via
+		(at 131 279)
+		(size 0.6)
+		(drill 0.3)
+		(layers "F.Cu" "B.Cu")
+		(free yes)
+		(net 5)
+	)
+	(via
+		(at 132 279)
+		(size 0.6)
+		(drill 0.3)
+		(layers "F.Cu" "B.Cu")
+		(free yes)
+		(net 5)
+	)
+	(via
 		(at 133.476891 42.874248)
 		(size 0.6)
@@
 	)
 	(via
+		(at 132 37)
+		(size 0.6)
+		(drill 0.3)
+		(layers "F.Cu" "B.Cu")
+		(free yes)
+		(net 5)
+	)
+	(via
+		(at 133 37)
+		(size 0.6)
+		(drill 0.3)
+		(layers "F.Cu" "B.Cu")
+		(free yes)
+		(net 5)
+	)
+	(via
 		(at 131.952891 42.874248)
 		(size 0.6)
@@
 		(drill 0.3)
 		(layers "F.Cu" "B.Cu")
+		(net 5)
+	)
+	(via
+		(at 131 37)
+		(size 0.6)
+		(drill 0.3)
+		(layers "F.Cu" "B.Cu")
+		(free yes)
+		(net 5)
+	)
+	(via
+		(at 134 37)
+		(size 0.6)
+		(drill 0.3)
+		(layers "F.Cu" "B.Cu")
+		(free yes)
+		(net 5)
+	)
+	(via
+		(at 133 279)
+		(size 0.6)
+		(drill 0.3)
+		(layers "F.Cu" "B.Cu")
+		(free yes)
+		(net 5)
+	)
+	(via
+		(at 133.5 247)
+		(size 0.6)
+		(drill 0.3)
+		(layers "F.Cu" "B.Cu")
+		(free yes)
 		(net 5)
 	)
@@
 	)
 	(segment
+		(start 128.725 262.015)
+		(end 127.575 260.865)
+		(width 0.2)
+		(layer "F.Cu")
+		(net 10)
+	)
+	(segment
+		(start 127.575 258.325)
+		(end 127 257.75)
+		(width 0.2)
+		(layer "F.Cu")
+		(net 10)
+	)
+	(segment
+		(start 129.875 243.125)
+		(end 129.875 233.165)
+		(width 0.2)
+		(layer "F.Cu")
+		(net 10)
+	)
+	(segment
 		(start 129.875 233.165)
 		(end 128.725 232.015)
@@
 	)
 	(segment
-		(start 127.508 246.734284)
-		(end 129.875 244.367284)
+		(start 127.575 260.865)
+		(end 127.575 258.325)
 		(width 0.2)
 		(layer "F.Cu")
@@
 	)
 	(segment
-		(start 127.508 260.798)
-		(end 127.508 246.734284)
+		(start 127 257.75)
+		(end 127 246)
 		(width 0.2)
 		(layer "F.Cu")
@@
 	)
 	(segment
-		(start 128.725 262.015)
-		(end 127.508 260.798)
-		(width 0.2)
-		(layer "F.Cu")
-		(net 10)
-	)
-	(segment
-		(start 129.875 244.367284)
-		(end 129.875 233.165)
-		(width 0.2)
-		(layer "F.Cu")
+		(start 127 246)
+		(end 129.875 243.125)
+		(width 0.2)
+		(layer "F.Cu")
